Commit message: 更新了末端执行器的模型

File: src/leonardo_description/psm_description/10_snake/00_snake_params.xacro (robot description, xacro)
@@ -3,47 +3,47 @@
 <robot xmlns:xacro="http://www.ros.org/wiki/xacro">
     <!-- ====================== 各连杆质量 m(kg) ====================== -->
-    <xacro:property name="link00_m" value="0.0258"/>
-    <xacro:property name="link01_m" value="0.00170"/>
-    <xacro:property name="link02_m" value="0.00170"/>
-    <xacro:property name="link03_m" value="0.0123"/>
-    <xacro:property name="link04_m" value="0.00170"/>
-    <xacro:property name="link05_m" value="0.00635"/>
-    <xacro:property name="link06_m" value="0.00170"/>
-    <xacro:property name="link07_m" value="0.00170"/>
-    <xacro:property name="link08_m" value="0.00170"/>
-    <xacro:property name="link09_m" value="0.00686"/>
-    <xacro:property name="link09b_m" value="0.000671"/>
-    <xacro:property name="link10_m" value="0.00619"/>
-    <xacro:property name="link11_m" value="0.00671"/>
-    <xacro:property name="link12_m" value="0.00671"/>
+    <xacro:property name="link00_m" value="0.0258" />
+    <xacro:property name="link01_m" value="0.00170" />
+    <xacro:property name="link02_m" value="0.00170" />
+    <xacro:property name="link03_m" value="0.0123" />
+    <xacro:property name="link04_m" value="0.00170" />
+    <xacro:property name="link05_m" value="0.00635" />
+    <xacro:property name="link06_m" value="0.00170" />
+    <xacro:property name="link07_m" value="0.00170" />
+    <xacro:property name="link08_m" value="0.00170" />
+    <xacro:property name="link09_m" value="0.00686" />
+    <xacro:property name="link09b_m" value="0.000671" />
+    <xacro:property name="link10_m" value="0.00619" />
+    <xacro:property name="link11_m" value="0.00671" />
+    <xacro:property name="link12_m" value="0.00671" />
     <!-- ====================== 各连杆外半径 r(m) ====================== -->
-    <xacro:property name="link00_r" value="0.004"/>
-    <xacro:property name="link01_r" value="0.004"/>
-    <xacro:property name="link02_r" value="0.004"/>
-    <xacro:property name="link03_r" value="0.004"/>
-    <xacro:property name="link04_r" value="0.004"/>
-    <xacro:property name="link05_r" value="0.004"/>
-    <xacro:property name="link06_r" value="0.004"/>
-    <xacro:property name="link07_r" value="0.004"/>
-    <xacro:property name="link08_r" value="0.004"/>
-    <xacro:property name="link09_r" value="0.004"/>
-    <xacro:property name="link09b_r" value="0.004"/>
-    <xacro:property name="link10_r" value="0.004"/>
-    <xacro:property name="link11_r" value="0.004"/>
-    <xacro:property name="link12_r" value="0.004"/>
+    <xacro:property name="link00_r" value="0.005" />
+    <xacro:property name="link01_r" value="0.005" />
+    <xacro:property name="link02_r" value="0.005" />
+    <xacro:property name="link03_r" value="0.005" />
+    <xacro:property name="link04_r" value="0.005" />
+    <xacro:property name="link05_r" value="0.005" />
+    <xacro:property name="link06_r" value="0.005" />
+    <xacro:property name="link07_r" value="0.005" />
+    <xacro:property name="link08_r" value="0.005" />
+    <xacro:property name="link09_r" value="0.005" />
+    <xacro:property name="link09b_r" value="0.005" />
+    <xacro:property name="link10_r" value="0.005" />
+    <xacro:property name="link11_r" value="0.005" />
+    <xacro:property name="link12_r" value="0.005" />
     <!-- ====================== 各连杆总长 l(m) ====================== -->
-    <xacro:property name="link00_l" value="0.05"/>
-    <xacro:property name="link01_l" value="0.0033"/>
-    <xacro:property name="link02_l" value="0.0033"/>
-    <xacro:property name="link03_l" value="0.0238"/>
-    <xacro:property name="link04_l" value="0.0033"/>
-    <xacro:property name="link05_l" value="0.0123"/>
-    <xacro:property name="link06_l" value="0.0033"/>
-    <xacro:property name="link07_l" value="0.0033"/>
-    <xacro:property name="link08_l" value="0.0033"/>
-    <xacro:property name="link09_l" value="0.0133"/>
-    <xacro:property name="link09b_l" value="0.0013"/>
-    <xacro:property name="link10_l" value="0.012"/>
-    <xacro:property name="link11_l" value="0.013"/>
-    <xacro:property name="link12_l" value="0.013"/>
+    <xacro:property name="link00_l" value="0.05" />
+    <xacro:property name="link01_l" value="0.0033" />
+    <xacro:property name="link02_l" value="0.0033" />
+    <xacro:property name="link03_l" value="0.0238" />
+    <xacro:property name="link04_l" value="0.0033" />
+    <xacro:property name="link05_l" value="0.0123" />
+    <xacro:property name="link06_l" value="0.0033" />
+    <xacro:property name="link07_l" value="0.0033" />
+    <xacro:property name="link08_l" value="0.0033" />
+    <xacro:property name="link09_l" value="0.0133" />
+    <xacro:property name="link09b_l" value="0.0013" />
+    <xacro:property name="link10_l" value="0.012" />
+    <xacro:property name="link11_l" value="0.013" />
+    <xacro:property name="link12_l" value="0.013" />
 </robot>

File: src/leonardo_description/psm_description/10_snake/69_snake_robot.xacro (robot description, xacro)
@@ -1,29 +1,29 @@
 <?xml version="1.0"?>
-<robot name="snake_robot" xmlns:xacro="http://www.ros.org/wiki/xacro">
+<robot xmlns:xacro="http://www.ros.org/wiki/xacro">
     <!--  00 加载 inertia 宏定义-->
-    <xacro:include filename="00_snake_inertia.xacro"/>
+    <xacro:include filename="00_snake_inertia.xacro" />
     <!-- 00 加载snake材质 -->
-    <xacro:include filename="00_snake_materials.xacro"/>
+    <xacro:include filename="00_snake_materials.xacro" />
     <!-- 11 stl模型缩1000倍，单位转为 米 -->
-    <xacro:property name="mesh_scale" value="0.001 0.001 0.001"/>
+    <xacro:property name="mesh_scale" value="0.001 0.001 0.001" />
     <!-- 12 stl模型路径 -->
-    <xacro:property name="stl_path" value="package://raphael_robot_description/meshes/snake"/>
+    <xacro:property name="stl_path" value="package://leonardo_description/psm_description/00_meshes/snake" />
     <!-- 13 各连杆的质量、外径、长度 -->
-    <xacro:include filename="00_snake_params.xacro"/>
+    <xacro:include filename="00_snake_params.xacro" />
     <!-- 14 创建连杆的函数 -->
-    <xacro:include filename="10_snake_links.xacro"/>
+    <xacro:include filename="10_snake_links.xacro" />
     <!-- 15 创建关节的函数 -->
-    <xacro:include filename="11_snake_joints.xacro"/>
+    <xacro:include filename="11_snake_joints.xacro" />
     <!-- 16 调用宏生成snake -->
-    <xacro:get_snake_links prefix="s1"/>
-    <xacro:get_snake_joints prefix="s1"/>
+    <xacro:get_snake_links prefix="s1" />
+    <xacro:get_snake_joints prefix="s1" />
     <!-- 17 生成 base_footprint_snake 固定基座 -->
-    <link name="base_footprint_snake"/>
+    <link name="base_footprint_snake" />
     <joint name="base_s1_link00" type="prismatic">
-        <parent link="base_footprint_snake"/>
-        <child link="s1_link00"/>
-        <origin xyz="0 0 0" rpy="0 0 0"/>
-        <axis xyz="1 0 0"/>
-        <limit lower="-0.1" upper="0.1" effort="1000" velocity="10"/>
+        <parent link="base_footprint_snake" />
+        <child link="s1_link00" />
+        <origin xyz="0 0 0" rpy="0 0 0" />
+        <axis xyz="1 0 0" />
+        <limit lower="-0.1" upper="0.1" effort="1000" velocity="10" />
     </joint>
 </robot>
