Commit message: 实现了简单的两齿轮啮合转动，一个固定，另一个公转+自转

File: src/leonardo_description/psm_description/10_snake/00_snake_materials.xacro (robot description, xacro)
@@ -1,273 +1,205 @@
 <?xml version="1.0" encoding="UTF-8"?>
-<!-- 全局材质库：3条连杆 × 22个编号，互不重叠色相段 -->
+<!-- 全局材质库：3条连杆 × 22个编号；17/19/20 白色，21/22 钳子同色 -->
 <robot xmlns:xacro="http://www.ros.org/wiki/xacro">
     <xacro:property name="alpha" value="1" />
-    <!-- ==================== 连杆1：红 → 黄（H 0° → 60°） ==================== -->
-    <!-- <material name="s1_link01">
-        <color rgba="0.950 0.143 0.143 ${alpha}" />
+    <!-- ==================== 连杆1：红橙黄暖色系 ==================== -->
+    <material name="s1_link01">
+        <color rgba="0.55 0.00 0.00 ${alpha}" />
     </material>
     <material name="s1_link02">
-        <color rgba="0.950 0.181 0.143 ${alpha}" />
+        <color rgba="0.75 0.05 0.00 ${alpha}" />
     </material>
     <material name="s1_link03">
-        <color rgba="0.950 0.219 0.143 ${alpha}" />
+        <color rgba="0.95 0.10 0.00 ${alpha}" />
     </material>
     <material name="s1_link04">
-        <color rgba="0.950 0.258 0.143 ${alpha}" />
+        <color rgba="1.00 0.20 0.00 ${alpha}" />
     </material>
     <material name="s1_link05">
-        <color rgba="0.950 0.296 0.143 ${alpha}" />
+        <color rgba="1.00 0.30 0.00 ${alpha}" />
     </material>
     <material name="s1_link06">
-        <color rgba="0.950 0.335 0.143 ${alpha}" />
+        <color rgba="1.00 0.40 0.00 ${alpha}" />
     </material>
     <material name="s1_link07">
-        <color rgba="0.950 0.373 0.143 ${alpha}" />
-    </material>
+        <color rgba="1.00 0.50 0.00 ${alpha}" />e </material>
     <material name="s1_link08">
-        <color rgba="0.950 0.412 0.143 ${alpha}" />
+        <color rgba="1.00 0.60 0.00 ${alpha}" />
     </material>
     <material name="s1_link09">
-        <color rgba="0.950 0.450 0.143 ${alpha}" />
+        <color rgba="1.00 0.70 0.00 ${alpha}" />
     </material>
     <material name="s1_link10">
-        <color rgba="0.950 0.489 0.143 ${alpha}" />
+        <color rgba="1.00 0.80 0.00 ${alpha}" />
     </material>
     <material name="s1_link11">
-        <color rgba="0.950 0.527 0.143 ${alpha}" />
+        <color rgba="1.00 0.90 0.00 ${alpha}" />
     </material>
     <material name="s1_link12">
-        <color rgba="0.950 0.565 0.143 ${alpha}" />
+        <color rgba="0.90 0.95 0.00 ${alpha}" />
     </material>
     <material name="s1_link13">
-        <color rgba="0.950 0.604 0.143 ${alpha}" />
+        <color rgba="0.80 0.40 0.00 ${alpha}" />
     </material>
     <material name="s1_link14">
-        <color rgba="0.950 0.642 0.143 ${alpha}" />
+        <color rgba="1.00 0.50 0.30 ${alpha}" />
     </material>
     <material name="s1_link15">
-        <color rgba="0.950 0.681 0.143 ${alpha}" />
+        <color rgba="1.00 0.60 0.40 ${alpha}" />
     </material>
     <material name="s1_link16">
-        <color rgba="0.950 0.719 0.143 ${alpha}" />
+        <color rgba="1.00 0.70 0.50 ${alpha}" />
     </material>
     <material name="s1_link17">
-        <color rgba="0.950 0.758 0.143 ${alpha}" />
+        <color rgba="1 1 1 ${alpha}" />
     </material>
     <material name="s1_link18">
-        <color rgba="0.950 0.796 0.143 ${alpha}" />
+        <color rgba="0.85 0.20 0.10 ${alpha}" />
     </material>
     <material name="s1_link19">
-        <color rgba="0.950 0.835 0.143 ${alpha}" />
+        <color rgba="1 1 1 ${alpha}" />
     </material>
     <material name="s1_link20">
-        <color rgba="0.950 0.873 0.143 ${alpha}" />
+        <color rgba="1 1 1 ${alpha}" />
     </material>
     <material name="s1_link21">
-        <color rgba="0.950 0.912 0.143 ${alpha}" />
+        <color rgba="0.85 0.00 0.45 ${alpha}" />
     </material>
     <material name="s1_link22">
-        <color rgba="0.950 0.950 0.143 ${alpha}" />
-    </material> -->
-    <!-- 最大对比度 -->
-    <material name="s1_link01">
-        <color rgba="0.3 0 0.5 ${alpha}" />
-    </material>
-    <material name="s1_link02">
-        <color rgba="1 0.6 0 ${alpha}" />
-    </material>
-    <material name="s1_link03">
-        <color rgba="0.3 0 0.5 ${alpha}" />
-    </material>
-    <material name="s1_link04">
-        <color rgba="1 0.6 0 ${alpha}" />
-    </material>
-    <material name="s1_link05">
-        <color rgba="0.3 0 0.5 ${alpha}" />
-    </material>
-    <material name="s1_link06">
-        <color rgba="1 0.6 0 ${alpha}" />
-    </material>
-    <material name="s1_link07">
-        <color rgba="0.3 0 0.5 ${alpha}" />
-    </material>
-    <material name="s1_link08">
-        <color rgba="1 0.6 0 ${alpha}" />
-    </material>
-    <material name="s1_link09">
-        <color rgba="0.3 0 0.5 ${alpha}" />
-    </material>
-    <material name="s1_link10">
-        <color rgba="1 0.6 0 ${alpha}" />
-    </material>
-    <material name="s1_link11">
-        <color rgba="0.3 0 0.5 ${alpha}" />
-    </material>
-    <material name="s1_link12">
-        <color rgba="1 0.6 0 ${alpha}" />
-    </material>
-    <material name="s1_link13">
-        <color rgba="0.3 0 0.5 ${alpha}" />
-    </material>
-    <material name="s1_link14">
-        <color rgba="1 0.6 0 ${alpha}" />
-    </material>
-    <material name="s1_link15">
-        <color rgba="0.3 0 0.5 ${alpha}" />
-    </material>
-    <material name="s1_link16">
-        <color rgba="1 0.6 0 ${alpha}" />
-    </material>
-    <material name="s1_link17">
-        <color rgba="0.3 0 0.5 ${alpha}" />
-    </material>
-    <material name="s1_link18">
-        <color rgba="1 0.6 0 ${alpha}" />
-    </material>
-    <material name="s1_link19">
-        <color rgba="0.3 0 0.5 ${alpha}" />
-    </material>
-    <material name="s1_link20">
-        <color rgba="1 0.6 0 ${alpha}" />
-    </material>
-    <material name="s1_link21">
-        <color rgba="0.3 0 0.5 ${alpha}" />
-    </material>
-    <material name="s1_link22">
-        <color rgba="1 0.6 0 ${alpha}" />
-    </material>
-    <!-- ==================== 连杆2：绿 → 青（H 120° → 180°） ==================== -->
+        <color rgba="0.85 0.00 0.45 ${alpha}" />
+    </material>
+    <!-- ==================== 连杆2：绿 → 青 ==================== -->
     <material name="s2_link01">
-        <color rgba="0.143 0.950 0.143 ${alpha}" />
+        <color rgba="0.00 0.35 0.00 ${alpha}" />
     </material>
     <material name="s2_link02">
-        <color rgba="0.143 0.950 0.181 ${alpha}" />
+        <color rgba="0.00 0.50 0.00 ${alpha}" />
     </material>
     <material name="s2_link03">
-        <color rgba="0.143 0.950 0.219 ${alpha}" />
+        <color rgba="0.00 0.65 0.00 ${alpha}" />
     </material>
     <material name="s2_link04">
-        <color rgba="0.143 0.950 0.258 ${alpha}" />
+        <color rgba="0.10 0.80 0.10 ${alpha}" />
     </material>
     <material name="s2_link05">
-        <color rgba="0.143 0.950 0.296 ${alpha}" />
+        <color rgba="0.00 0.90 0.20 ${alpha}" />
     </material>
     <material name="s2_link06">
-        <color rgba="0.143 0.950 0.335 ${alpha}" />
+        <color rgba="0.00 1.00 0.35 ${alpha}" />
     </material>
     <material name="s2_link07">
-        <color rgba="0.143 0.950 0.373 ${alpha}" />
+        <color rgba="0.00 0.85 0.50 ${alpha}" />
     </material>
     <material name="s2_link08">
-        <color rgba="0.143 0.950 0.412 ${alpha}" />
+        <color rgba="0.00 0.75 0.60 ${alpha}" />
     </material>
     <material name="s2_link09">
-        <color rgba="0.143 0.950 0.450 ${alpha}" />
+        <color rgba="0.00 0.90 0.75 ${alpha}" />
     </material>
     <material name="s2_link10">
-        <color rgba="0.143 0.950 0.489 ${alpha}" />
+        <color rgba="0.00 0.80 0.90 ${alpha}" />
     </material>
     <material name="s2_link11">
-        <color rgba="0.143 0.950 0.527 ${alpha}" />
+        <color rgba="0.00 0.60 0.90 ${alpha}" />
     </material>
     <material name="s2_link12">
-        <color rgba="0.143 0.950 0.565 ${alpha}" />
+        <color rgba="0.00 0.95 1.00 ${alpha}" />
     </material>
     <material name="s2_link13">
-        <color rgba="0.143 0.950 0.604 ${alpha}" />
+        <color rgba="0.20 0.70 0.50 ${alpha}" />
     </material>
     <material name="s2_link14">
-        <color rgba="0.143 0.950 0.642 ${alpha}" />
+        <color rgba="0.30 0.85 0.70 ${alpha}" />
     </material>
     <material name="s2_link15">
-        <color rgba="0.143 0.950 0.681 ${alpha}" />
+        <color rgba="0.50 0.95 0.80 ${alpha}" />
     </material>
     <material name="s2_link16">
-        <color rgba="0.143 0.950 0.719 ${alpha}" />
+        <color rgba="0.60 0.80 0.20 ${alpha}" />
     </material>
     <material name="s2_link17">
-        <color rgba="0.143 0.950 0.758 ${alpha}" />
+        <color rgba="1 1 1 ${alpha}" />
     </material>
     <material name="s2_link18">
-        <color rgba="0.143 0.950 0.796 ${alpha}" />
+        <color rgba="0.10 0.55 0.35 ${alpha}" />
     </material>
     <material name="s2_link19">
-        <color rgba="0.143 0.950 0.835 ${alpha}" />
+        <color rgba="1 1 1 ${alpha}" />
     </material>
     <material name="s2_link20">
-        <color rgba="0.143 0.950 0.873 ${alpha}" />
+        <color rgba="1 1 1 ${alpha}" />
     </material>
     <material name="s2_link21">
-        <color rgba="0.143 0.950 0.912 ${alpha}" />
+        <color rgba="0.00 0.75 0.85 ${alpha}" />
     </material>
     <material name="s2_link22">
-        <color rgba="0.143 0.950 0.950 ${alpha}" />
-    </material>
-    <!-- ==================== 连杆3：蓝 → 紫（H 240° → 300°） ==================== -->
+        <color rgba="0.00 0.75 0.85 ${alpha}" />
+    </material>
+    <!-- ==================== 连杆3：蓝 → 紫 ==================== -->
     <material name="s3_link01">
-        <color rgba="0.143 0.143 0.950 ${alpha}" />
+        <color rgba="0.00 0.00 0.45 ${alpha}" />
     </material>
     <material name="s3_link02">
-        <color rgba="0.181 0.143 0.950 ${alpha}" />
+        <color rgba="0.00 0.00 0.60 ${alpha}" />
     </material>
     <material name="s3_link03">
-        <color rgba="0.219 0.143 0.950 ${alpha}" />
+        <color rgba="0.00 0.00 0.80 ${alpha}" />
     </material>
     <material name="s3_link04">
-        <color rgba="0.258 0.143 0.950 ${alpha}" />
+        <color rgba="0.10 0.10 0.95 ${alpha}" />
     </material>
     <material name="s3_link05">
-        <color rgba="0.296 0.143 0.950 ${alpha}" />
+        <color rgba="0.20 0.20 0.90 ${alpha}" />
     </material>
     <material name="s3_link06">
-        <color rgba="0.335 0.143 0.950 ${alpha}" />
+        <color rgba="0.30 0.30 0.95 ${alpha}" />
     </material>
     <material name="s3_link07">
-        <color rgba="0.373 0.143 0.950 ${alpha}" />
+        <color rgba="0.40 0.20 0.90 ${alpha}" />
     </material>
     <material name="s3_link08">
-        <color rgba="0.412 0.143 0.950 ${alpha}" />
+        <color rgba="0.50 0.10 0.85 ${alpha}" />
     </material>
     <material name="s3_link09">
-        <color rgba="0.450 0.143 0.950 ${alpha}" />
+        <color rgba="0.60 0.10 0.80 ${alpha}" />
     </material>
     <material name="s3_link10">
-        <color rgba="0.489 0.143 0.950 ${alpha}" />
+        <color rgba="0.70 0.00 0.70 ${alpha}" />
     </material>
     <material name="s3_link11">
-        <color rgba="0.527 0.143 0.950 ${alpha}" />
+        <color rgba="0.80 0.00 0.60 ${alpha}" />
     </material>
     <material name="s3_link12">
-        <color rgba="0.565 0.143 0.950 ${alpha}" />
+        <color rgba="0.90 0.00 0.50 ${alpha}" />
     </material>
     <material name="s3_link13">
-        <color rgba="0.604 0.143 0.950 ${alpha}" />
+        <color rgba="0.50 0.00 0.50 ${alpha}" />
     </material>
     <material name="s3_link14">
-        <color rgba="0.642 0.143 0.950 ${alpha}" />
+        <color rgba="0.75 0.25 0.75 ${alpha}" />
     </material>
     <material name="s3_link15">
-        <color rgba="0.681 0.143 0.950 ${alpha}" />
+        <color rgba="0.85 0.40 0.85 ${alpha}" />
     </material>
     <material name="s3_link16">
-        <color rgba="0.719 0.143 0.950 ${alpha}" />
+        <color rgba="0.95 0.60 0.95 ${alpha}" />
     </material>
     <material name="s3_link17">
-        <color rgba="0.758 0.143 0.950 ${alpha}" />
+        <color rgba="1 1 1 ${alpha}" />
     </material>
     <material name="s3_link18">
-        <color rgba="0.796 0.143 0.950 ${alpha}" />
+        <color rgba="0.20 0.30 0.75 ${alpha}" />
     </material>
     <material name="s3_link19">
-        <color rgba="0.835 0.143 0.950 ${alpha}" />
+        <color rgba="1 1 1 ${alpha}" />
     </material>
     <material name="s3_link20">
-        <color rgba="0.873 0.143 0.950 ${alpha}" />
+        <color rgba="1 1 1 ${alpha}" />
     </material>
     <material name="s3_link21">
-        <color rgba="0.912 0.143 0.950 ${alpha}" />
+        <color rgba="0.65 0.00 0.95 ${alpha}" />
     </material>
     <material name="s3_link22">
-        <color rgba="0.950 0.143 0.950 ${alpha}" />
+        <color rgba="0.65 0.00 0.95 ${alpha}" />
     </material>
 </robot>

File: src/leonardo_description/psm_description/10_snake/00_snake_params.xacro (robot description, xacro)
@@ -68,6 +68,6 @@
     <xacro:property name="link18_l" value="0.0033" />
     <xacro:property name="link19_l" value="0.0133" />
-    <xacro:property name="link20_l" value="0.012" />
-    <xacro:property name="link21_l" value="0.013" />
-    <xacro:property name="link22_l" value="0.013" />
+    <xacro:property name="link20_l" value="0.0033" />
+    <xacro:property name="link21_l" value="0.0033" />
+    <xacro:property name="link22_l" value="0.0133" />
 </robot>

File: src/leonardo_description/psm_description/10_snake/10_snake_links.xacro (robot description, xacro)
@@ -26,5 +26,5 @@
                     <mesh filename="${stl_path}/02.stl" scale="${mesh_scale}" />
                 </geometry>
-                <origin xyz="0 0 0" rpy="0 0 0" />
+                <origin xyz="0 0 0" rpy="${pi} 0 0" />
                 <material name="${prefix}_link02" />
             </visual>
@@ -116,5 +116,5 @@
                     <mesh filename="${stl_path}/07.stl" scale="${mesh_scale}" />
                 </geometry>
-                <origin xyz="0 0 0" rpy="0 0 0" />
+                <origin xyz="0 0 0" rpy="${pi} 0 0" />
                 <material name="${prefix}_link07" />
             </visual>
@@ -134,5 +134,5 @@
                     <mesh filename="${stl_path}/08.stl" scale="${mesh_scale}" />
                 </geometry>
-                <origin xyz="0 0 0" rpy="0 0 0" />
+                <origin xyz="0 0 0" rpy="${pi} ${pi/2.0} 0" />
                 <material name="${prefix}_link08" />
             </visual>
@@ -152,5 +152,5 @@
                     <mesh filename="${stl_path}/09.stl" scale="${mesh_scale}" />
                 </geometry>
-                <origin xyz="0 0 0" rpy="0 0 0" />
+                <origin xyz="0 0 0" rpy="${pi} 0 0" />
                 <material name="${prefix}_link09" />
             </visual>
@@ -206,5 +206,5 @@
                     <mesh filename="${stl_path}/12.stl" scale="${mesh_scale}" />
                 </geometry>
-                <origin xyz="0 0 0" rpy="0 0 0" />
+                <origin xyz="0 0 0" rpy="0 ${pi/2.0} 0" />
                 <material name="${prefix}_link12" />
             </visual>
@@ -242,5 +242,5 @@
                     <mesh filename="${stl_path}/14.stl" scale="${mesh_scale}" />
                 </geometry>
-                <origin xyz="0 0 0" rpy="0 0 0" />
+                <origin xyz="0 0 0" rpy="0 ${pi/2.0} 0" />
                 <material name="${prefix}_link14" />
             </visual>
@@ -296,5 +296,5 @@
                     <mesh filename="${stl_path}/17.stl" scale="${mesh_scale}" />
                 </geometry>
-                <origin xyz="0 0 0" rpy="0 0 0" />
+                <origin xyz="0 0 0" rpy="0 0 ${pi/2.0}" />
                 <material name="${prefix}_link17" />
             </visual>
@@ -314,5 +314,5 @@
                     <mesh filename="${stl_path}/18.stl" scale="${mesh_scale}" />
                 </geometry>
-                <origin xyz="0 0 0" rpy="0 0 0" />
+                <origin xyz="0 0 0" rpy="0 0 ${pi}" />
                 <material name="${prefix}_link18" />
             </visual>
@@ -332,5 +332,5 @@
                     <mesh filename="${stl_path}/19.stl" scale="${mesh_scale}" />
                 </geometry>
-                <origin xyz="0 0 0" rpy="0 0 0" />
+                <origin xyz="0 0 0" rpy="${pi/2.0} 0 0" />
                 <material name="${prefix}_link19" />
             </visual>
@@ -350,5 +350,5 @@
                     <mesh filename="${stl_path}/20.stl" scale="${mesh_scale}" />
                 </geometry>
-                <origin xyz="0 0 0" rpy="0 0 0" />
+                <origin xyz="0 0 -0.004" rpy="${pi/2.0} 0 0" />
                 <material name="${prefix}_link20" />
             </visual>
@@ -368,5 +368,5 @@
                     <mesh filename="${stl_path}/21.stl" scale="${mesh_scale}" />
                 </geometry>
-                <origin xyz="0 0 0" rpy="0 0 0" />
+                <origin xyz="0 0 0" rpy="${pi/2.0} 0 0" />
                 <material name="${prefix}_link21" />
             </visual>
@@ -386,5 +386,5 @@
                     <mesh filename="${stl_path}/22.stl" scale="${mesh_scale}" />
                 </geometry>
-                <origin xyz="0 0 0" rpy="0 0 0" />
+                <origin xyz="0 0 0" rpy="${pi/2.0} ${pi} 0" />
                 <material name="${prefix}_link22" />
             </visual>
