Commit message: 实现了简单的两齿轮啮合转动，一个固定，另一个公转+自转

File: src/leonardo_description/psm_description/10_snake/11_snake_joints.xacro (robot description, xacro)
@@ -3,50 +3,42 @@
 <robot xmlns:xacro="http://www.ros.org/wiki/xacro">
     <!-- ==========  X 轴偏移量  ========== -->
-    <xacro:property name="x_offset_01_02" value="0.001" />
-    <xacro:property name="x_offset_02_03" value="0.05" />
-    <xacro:property name="x_offset_03_04" value="0.004" />
-    <xacro:property name="x_offset_04_05" value="0.004" />
-    <xacro:property name="x_offset_05_06" value="0.01" />
-    <xacro:property name="x_offset_06_07" value="0.03" />
-    <xacro:property name="x_offset_07_08" value="0.01" />
-    <xacro:property name="x_offset_08_09" value="0.01" />
-    <xacro:property name="x_offset_09_10" value="0.01" />
-    <xacro:property name="x_offset_10_11" value="0.01" />
-    <xacro:property name="x_offset_10_12" value="0.01" />
-    <xacro:property name="x_offset_12_13" value="0.01" />
-    <xacro:property name="x_offset_13_14" value="0.02" />
-    <xacro:property name="x_offset_14_15" value="0.02" />
-    <xacro:property name="x_offset_15_16" value="0.02" />
-    <xacro:property name="x_offset_16_17" value="0.02" />
-    <xacro:property name="x_offset_17_18" value="0.02" />
-    <xacro:property name="x_offset_18_19" value="0.02" />
-    <xacro:property name="x_offset_19_20" value="0.01" />
-    <xacro:property name="x_offset_20_21" value="0.01" />
-    <xacro:property name="x_offset_21_22" value="0.01" />
+    <xacro:property name="y_offset_01_02" value="0.051" />
+    <xacro:property name="y_offset_02_03" value="0.001" />
+    <xacro:property name="y_offset_03_04" value="0.004" />
+    <xacro:property name="y_offset_04_05" value="0.004" />
+    <xacro:property name="y_offset_05_06" value="0.0084" />
+    <xacro:property name="y_offset_06_07" value="0.0084" />
+    <xacro:property name="y_offset_07_08" value="0.004" />
+    <xacro:property name="y_offset_08_09" value="0.004" />
+    <xacro:property name="y_offset_09_10" value="0.0055" />
+    <xacro:property name="y_offset_10_11" value="0.0" />
+    <xacro:property name="y_offset_11_12" value="0.004" />
+    <xacro:property name="y_offset_12_13" value="0.004" />
+    <xacro:property name="y_offset_13_14" value="0.004" />
+    <xacro:property name="y_offset_14_15" value="0.004" />
+    <xacro:property name="y_offset_15_16" value="0.0015" />
+    <xacro:property name="y_offset_16_17" value="0.01172" />
+    <xacro:property name="y_offset_17_18" value="0.00728" />
+    <xacro:property name="y_offset_18_19" value="-0.0013" />
+    <xacro:property name="y_offset_19_20" value="0.005" />
+    <xacro:property name="y_offset_20_21" value="0.0" />
+    <xacro:property name="y_offset_20_22" value="0.0" />
     <!-- ========= 最大力矩 ======== -->
     <xacro:property name="effort" value="1000" />
     <!-- ========= 最大速度 rad/s ======== -->
     <xacro:property name="velocity" value="${4.0 * pi}" />
-    <!-- ========= 旋转角度 /度 ======== -->
-    <xacro:property name="rad_30" value="${30 * pi / 180.0}" />
-    <xacro:property name="rad_135" value="${135 * pi / 180.0}" />
-    <xacro:property name="rad_fork" value="${30 * pi / 180.0}" />
     <!-- ========== 宏定义：生成所有关节 ========== -->
     <xacro:macro name="get_snake_joints" params="prefix">
         <!-- link01 -> link02 -->
-        <joint name="${prefix}_joint_01_02" type="revolute">
+        <joint name="${prefix}_joint_01_02" type="fixed">
             <parent link="${prefix}_01" />
             <child link="${prefix}_02" />
-            <origin xyz="0 ${x_offset_01_02} 0" rpy="0 0 0" />
-            <axis xyz="0 1 0" />
-            <limit effort="${effort}" velocity="${velocity}" lower="${-rad_30}" upper="${rad_30}" />
+            <origin xyz="0 ${y_offset_01_02} 0" rpy="0 0 0" />
         </joint>
         <!-- link02 -> link03 -->
-        <joint name="${prefix}_joint_02_03" type="revolute">
+        <joint name="${prefix}_joint_02_03" type="fixed">
             <parent link="${prefix}_02" />
             <child link="${prefix}_03" />
-            <origin xyz="0 ${x_offset_02_03} 0" rpy="0 0 0" />
-            <axis xyz="0 0 1" />
-            <limit effort="${effort}" velocity="${velocity}" lower="${-rad_30}" upper="${rad_30}" />
+            <origin xyz="0 ${y_offset_02_03} 0" rpy="0 0 0" />
         </joint>
         <!-- link03 -> link04 -->
@@ -54,7 +46,7 @@
             <parent link="${prefix}_03" />
             <child link="${prefix}_04" />
-            <origin xyz="0 ${x_offset_03_04} 0" rpy="0 0 0" />
+            <origin xyz="0 ${y_offset_03_04} 0" rpy="0 0 0" />
             <axis xyz="0 0 1" />
-            <limit effort="${effort}" velocity="${velocity}" lower="${-rad_30}" upper="${rad_30}" />
+            <limit effort="${effort}" velocity="${velocity}" lower="${-pi}" upper="${pi}" />
         </joint>
         <!-- link04 -> link05 -->
@@ -62,23 +54,19 @@
             <parent link="${prefix}_04" />
             <child link="${prefix}_05" />
-            <origin xyz="0 ${x_offset_04_05} 0" rpy="0 0 0" />
-            <axis xyz="0 1 0" />
-            <limit effort="${effort}" velocity="${velocity}" lower="${-rad_30}" upper="${rad_30}" />
+            <origin xyz="0 ${y_offset_04_05} 0" rpy="0 0 0" />
+            <axis xyz="1 0 0" />
+            <limit effort="${effort}" velocity="${velocity}" lower="${-pi}" upper="${pi}" />
         </joint>
         <!-- link05 -> link06 -->
-        <joint name="${prefix}_joint_05_06" type="revolute">
+        <joint name="${prefix}_joint_05_06" type="fixed">
             <parent link="${prefix}_05" />
             <child link="${prefix}_06" />
-            <origin xyz="0 ${x_offset_05_06} 0" rpy="0 0 0" />
-            <axis xyz="0 1 0" />
-            <limit effort="${effort}" velocity="${velocity}" lower="${-rad_30}" upper="${rad_30}" />
+            <origin xyz="0 ${y_offset_05_06} 0" rpy="0 0 0" />
         </joint>
         <!-- link06 -> link07 -->
-        <joint name="${prefix}_joint_06_07" type="revolute">
+        <joint name="${prefix}_joint_06_07" type="fixed">
             <parent link="${prefix}_06" />
             <child link="${prefix}_07" />
-            <origin xyz="0 ${x_offset_06_07} 0" rpy="0 0 0" />
-            <axis xyz="0 0 1" />
-            <limit effort="${effort}" velocity="${velocity}" lower="${-rad_30}" upper="${rad_30}" />
+            <origin xyz="0 ${y_offset_06_07} 0" rpy="0 0 0" />
         </joint>
         <!-- link07 -> link08 -->
@@ -86,7 +74,7 @@
             <parent link="${prefix}_07" />
             <child link="${prefix}_08" />
-            <origin xyz="0 ${x_offset_07_08} 0" rpy="0 0 0" />
-            <axis xyz="0 1 0" />
-            <limit effort="${effort}" velocity="${velocity}" lower="${-rad_30}" upper="${rad_30}" />
+            <origin xyz="0 ${y_offset_07_08} 0" rpy="0 0 0" />
+            <axis xyz="1 0 0" />
+            <limit effort="${effort}" velocity="${velocity}" lower="${-pi}" upper="${pi}" />
         </joint>
         <!-- link08 -> link09 -->
@@ -94,32 +82,27 @@
             <parent link="${prefix}_08" />
             <child link="${prefix}_09" />
-            <origin xyz="0 ${x_offset_08_09} 0" rpy="0 0 0" />
+            <origin xyz="0 ${y_offset_08_09} 0" rpy="0 0 0" />
             <axis xyz="0 0 1" />
-            <limit effort="${effort}" velocity="${velocity}" lower="${-rad_30}" upper="${rad_30}" />
+            <limit effort="${effort}" velocity="${velocity}" lower="${-pi}" upper="${pi}" />
         </joint>
-        <!-- link09 -> link10 （合并原 link09b 固定关节与旋转关节） -->
-        <joint name="${prefix}_joint_09_10" type="revolute">
+        <!-- link09 -> link10  -->
+        <joint name="${prefix}_joint_09_10" type="fixed">
             <parent link="${prefix}_09" />
             <child link="${prefix}_10" />
-            <origin xyz="0 ${x_offset_09_10} 0" rpy="0 0 0" />
-            <axis xyz="1 0 0" />
-            <limit effort="${effort}" velocity="${velocity}" lower="${-rad_135}" upper="${rad_135}" />
+            <origin xyz="0 ${y_offset_09_10} 0" rpy="0 0 0" />
         </joint>
-        <!-- link10 -> link11 【主动驱动关节，电机驱动】 -->
-        <joint name="${prefix}_joint_10_11" type="revolute">
+        <!-- link10 -> link11  -->
+        <joint name="${prefix}_joint_10_11" type="fixed">
             <parent link="${prefix}_10" />
             <child link="${prefix}_11" />
-            <origin xyz="0 ${x_offset_10_11} 0" rpy="0 0 0" />
-            <axis xyz="0 1 0" />
-            <limit effort="${effort}" velocity="${velocity}" lower="${-rad_fork}" upper="0" />
+            <origin xyz="0 ${y_offset_10_11} 0" rpy="0 0 0" />
         </joint>
-        <!-- link10 -> link12 【mimic镜像跟随，剪刀另一侧刀片】 -->
-        <joint name="${prefix}_joint_10_12" type="revolute">
-            <parent link="${prefix}_10" />
+        <!-- link11 -> link12  -->
+        <joint name="${prefix}_joint_11_12" type="revolute">
+            <parent link="${prefix}_11" />
             <child link="${prefix}_12" />
-            <origin xyz="0 ${x_offset_10_12} 0" rpy="0 0 0" />
-            <axis xyz="0 1 0" />
-            <limit effort="${effort}" velocity="${velocity}" lower="0" upper="${rad_fork}" />
-            <mimic joint="${prefix}_joint_10_11" multiplier="-1.0" offset="0.0" />
+            <origin xyz="0 ${y_offset_11_12} 0" rpy="0 0 0" />
+            <axis xyz="0 0 1" />
+            <limit effort="${effort}" velocity="${velocity}" lower="${-pi}" upper="${pi}" />
         </joint>
         <!-- link12 -> link13 -->
@@ -127,7 +110,7 @@
             <parent link="${prefix}_12" />
             <child link="${prefix}_13" />
-            <origin xyz="0 ${x_offset_12_13} 0" rpy="0 0 0" />
-            <axis xyz="0 1 0" />
-            <limit effort="${effort}" velocity="${velocity}" lower="${-rad_30}" upper="${rad_30}" />
+            <origin xyz="0 ${y_offset_12_13} 0" rpy="0 0 0" />
+            <axis xyz="1 0 0" />
+            <limit effort="${effort}" velocity="${velocity}" lower="${-pi}" upper="${pi}" />
         </joint>
         <!-- link13 -> link14 -->
@@ -135,7 +118,7 @@
             <parent link="${prefix}_13" />
             <child link="${prefix}_14" />
-            <origin xyz="0 ${x_offset_13_14} 0" rpy="0 0 0" />
+            <origin xyz="0 ${y_offset_13_14} 0" rpy="0 0 0" />
             <axis xyz="0 0 1" />
-            <limit effort="${effort}" velocity="${velocity}" lower="${-rad_30}" upper="${rad_30}" />
+            <limit effort="${effort}" velocity="${velocity}" lower="${-pi}" upper="${pi}" />
         </joint>
         <!-- link14 -> link15 -->
@@ -143,23 +126,19 @@
             <parent link="${prefix}_14" />
             <child link="${prefix}_15" />
-            <origin xyz="0 ${x_offset_14_15} 0" rpy="0 0 0" />
-            <axis xyz="0 1 0" />
-            <limit effort="${effort}" velocity="${velocity}" lower="${-rad_30}" upper="${rad_30}" />
+            <origin xyz="0 ${y_offset_14_15} 0" rpy="0 0 0" />
+            <axis xyz="1 0 0" />
+            <limit effort="${effort}" velocity="${velocity}" lower="${-pi}" upper="${pi}" />
         </joint>
         <!-- link15 -> link16 -->
-        <joint name="${prefix}_joint_15_16" type="revolute">
+        <joint name="${prefix}_joint_15_16" type="fixed">
             <parent link="${prefix}_15" />
             <child link="${prefix}_16" />
-            <origin xyz="0 ${x_offset_15_16} 0" rpy="0 0 0" />
-            <axis xyz="0 1 0" />
-            <limit effort="${effort}" velocity="${velocity}" lower="${-rad_30}" upper="${rad_30}" />
+            <origin xyz="0 ${y_offset_15_16} 0" rpy="0 0 0" />
         </joint>
         <!-- link16 -> link17 -->
-        <joint name="${prefix}_joint_16_17" type="revolute">
+        <joint name="${prefix}_joint_16_17" type="fixed">
             <parent link="${prefix}_16" />
             <child link="${prefix}_17" />
-            <origin xyz="0 ${x_offset_16_17} 0" rpy="0 0 0" />
-            <axis xyz="0 0 1" />
-            <limit effort="${effort}" velocity="${velocity}" lower="${-rad_30}" upper="${rad_30}" />
+            <origin xyz="0 ${y_offset_16_17} 0" rpy="0 0 0" />
         </joint>
         <!-- link17 -> link18 -->
@@ -167,39 +146,35 @@
             <parent link="${prefix}_17" />
             <child link="${prefix}_18" />
-            <origin xyz="0 ${x_offset_17_18} 0" rpy="0 0 0" />
+            <origin xyz="0 ${y_offset_17_18} 0" rpy="0 0 0" />
             <axis xyz="0 1 0" />
-            <limit effort="${effort}" velocity="${velocity}" lower="${-rad_30}" upper="${rad_30}" />
+            <limit effort="${effort}" velocity="${velocity}" lower="${-pi}" upper="${pi}" />
         </joint>
         <!-- link18 -> link19 -->
-        <joint name="${prefix}_joint_18_19" type="revolute">
+        <joint name="${prefix}_joint_18_19" type="fixed">
             <parent link="${prefix}_18" />
             <child link="${prefix}_19" />
-            <origin xyz="0 ${x_offset_18_19} 0" rpy="0 0 0" />
-            <axis xyz="0 0 1" />
-            <limit effort="${effort}" velocity="${velocity}" lower="${-rad_30}" upper="${rad_30}" />
+            <origin xyz="0 ${y_offset_18_19} 0" rpy="0 0 0" />
         </joint>
         <!-- link19 -> link20 -->
-        <joint name="${prefix}_joint_19_20" type="revolute">
+        <joint name="${prefix}_joint_19_20" type="fixed">
             <parent link="${prefix}_19" />
             <child link="${prefix}_20" />
-            <origin xyz="0 ${x_offset_19_20} 0" rpy="0 0 0" />
-            <axis xyz="1 0 0" />
-            <limit effort="${effort}" velocity="${velocity}" lower="${-rad_135}" upper="${rad_135}" />
+            <origin xyz="0 ${y_offset_19_20} 0" rpy="0 0 0" />
         </joint>
-        <!-- link20 -> link21 【主动驱动关节】 -->
+        <!-- link20 -> link21 （主动钳） -->
         <joint name="${prefix}_joint_20_21" type="revolute">
             <parent link="${prefix}_20" />
             <child link="${prefix}_21" />
-            <origin xyz="0 ${x_offset_20_21} 0" rpy="0 0 0" />
-            <axis xyz="0 1 0" />
-            <limit effort="${effort}" velocity="${velocity}" lower="${-rad_fork}" upper="0" />
+            <origin xyz="0 ${y_offset_20_21} 0" rpy="0 0 0" />
+            <axis xyz="0 0 1" />
+            <limit effort="${effort}" velocity="${velocity}" lower="0" upper="${pi/3.0}" />
         </joint>
-        <!-- link21 -> link22 【mimic镜像跟随】 -->
-        <joint name="${prefix}_joint_21_22" type="revolute">
-            <parent link="${prefix}_21" />
+        <!-- link20 -> link22 （镜像钳） -->
+        <joint name="${prefix}_joint_20_22" type="revolute">
+            <parent link="${prefix}_20" />
             <child link="${prefix}_22" />
-            <origin xyz="0 ${x_offset_21_22} 0" rpy="0 0 0" />
-            <axis xyz="0 1 0" />
-            <limit effort="${effort}" velocity="${velocity}" lower="0" upper="${rad_fork}" />
+            <origin xyz="0 ${y_offset_20_22} 0" rpy="0 0 0" />
+            <axis xyz="0 0 1" />
+            <limit effort="${effort}" velocity="${velocity}" lower="${-pi/3.0}" upper="${0}" />
             <mimic joint="${prefix}_joint_20_21" multiplier="-1.0" offset="0.0" />
         </joint>

File: src/leonardo_description/psm_description/10_snake/69_snake_robot.xacro (robot description, xacro)
@@ -15,15 +15,27 @@
     <!-- 15 创建关节的函数 -->
     <xacro:include filename="11_snake_joints.xacro" />
-    <!-- 16 调用宏生成snake -->
+    <!-- 16 调用宏生成3条snake和jonints -->
     <xacro:get_snake_links prefix="s1" />
+    <xacro:get_snake_links prefix="s2" />
+    <xacro:get_snake_links prefix="s3" />
     <xacro:get_snake_joints prefix="s1" />
+    <xacro:get_snake_joints prefix="s2" />
+    <xacro:get_snake_joints prefix="s3" />
     <!-- 17 生成 base_footprint_snake 固定基座 -->
     <link name="base_footprint_snake" />
-    <joint name="base_s1_link01" type="prismatic">
+    <joint name="base_s1_link01" type="fixed">
         <parent link="base_footprint_snake" />
         <child link="s1_01" />
         <origin xyz="0 0 0" rpy="0 0 0" />
-        <axis xyz="1 0 0" />
-        <limit lower="-0.1" upper="0.1" effort="1000" velocity="10" />
+    </joint>
+    <joint name="base_s2_link01" type="fixed">
+        <parent link="base_footprint_snake" />
+        <child link="s2_01" />
+        <origin xyz="0.05 0 0" rpy="0 0 0" />
+    </joint>
+    <joint name="base_s3_link01" type="fixed">
+        <parent link="base_footprint_snake" />
+        <child link="s3_01" />
+        <origin xyz="-0.05 0 0" rpy="0 0 0" />
     </joint>
 </robot>
