Commit message: intelligent_can已搭好了hardware, controller的架构，具体内容还没填。  description里面，4个虚拟电机也搞好了

File: src/leonardo_description/psm_description/10_snake/10_snake_links.xacro (robot description, xacro)
@@ -2,4 +2,9 @@
 <robot xmlns:xacro="http://www.ros.org/wiki/xacro">
     <xacro:macro name="get_snake_links" params="prefix">
+        <!-- ==================== 4个虚拟link，用来生成4个虚拟旋转joint ==================== -->
+        <link name="${prefix}_link_for_motor_01" />
+        <link name="${prefix}_link_for_motor_02" />
+        <link name="${prefix}_link_for_motor_03" />
+        <link name="${prefix}_link_for_motor_04" />
         <!-- ==================== Link 01 ==================== -->
         <link name="${prefix}_01">

File: src/leonardo_description/psm_description/10_snake/11_snake_joints.xacro (robot description, xacro)
@@ -44,4 +44,33 @@
     <!-- ========== 宏定义：生成所有关节 ========== -->
     <xacro:macro name="get_snake_joints" params="prefix">
+        <!-- ****************************************  4个虚拟旋转joint  **************************************** -->
+        <joint name="${prefix}_joint_motor_01" type="revolute">
+            <parent link="${prefix}_01" />
+            <child link="${prefix}_link_for_motor_01" />
+            <origin xyz="0 0 0.01" rpy="0 0 0" />
+            <axis xyz="0 0 1" />
+            <limit effort="${effort}" velocity="${velocity}" lower="${-pi/2.0}" upper="${pi/2.0}" />
+        </joint>
+        <joint name="${prefix}_joint_motor_02" type="revolute">
+            <parent link="${prefix}_01" />
+            <child link="${prefix}_link_for_motor_02" />
+            <origin xyz="0.005 0 0.01" rpy="0 0 0" />
+            <axis xyz="0 0 1" />
+            <limit effort="${effort}" velocity="${velocity}" lower="${-pi/2.0}" upper="${pi/2.0}" />
+        </joint>
+        <joint name="${prefix}_joint_motor_03" type="revolute">
+            <parent link="${prefix}_01" />
+            <child link="${prefix}_link_for_motor_03" />
+            <origin xyz="0.01 0 0.01" rpy="0 0 0" />
+            <axis xyz="0 0 1" />
+            <limit effort="${effort}" velocity="${velocity}" lower="${-pi/2.0}" upper="${pi/2.0}" />
+        </joint>
+        <joint name="${prefix}_joint_motor_04" type="revolute">
+            <parent link="${prefix}_01" />
+            <child link="${prefix}_link_for_motor_04" />
+            <origin xyz="0.015 0 0.01" rpy="0 0 0" />
+            <axis xyz="0 0 1" />
+            <limit effort="${effort}" velocity="${velocity}" lower="${-pi/2.0}" upper="${pi/2.0}" />
+        </joint>
         <!-- ****************************************  link01 -> link02  **************************************** -->
         <joint name="${prefix}_joint_01_02" type="fixed">

File: src/leonardo_description/psm_description/10_snake/88_snake_robot.ros2_control.xacro (robot description, xacro)
@@ -1,7 +1,7 @@
 <?xml version="1.0"?>
 <robot xmlns:xacro="http://www.ros.org/wiki/xacro">
-    <ros2_control name="PSMCan0Hardware" type="system">
+    <ros2_control name="IntelligentCan0Ros2Control" type="system">
         <hardware>
-            <plugin>psm_can_hardware/PSMCan0HardwareInterface</plugin>
+            <plugin>psm_hardware_interface/IntelligentCan0HardwareInterface</plugin>
             <!-- CAN 通道 -->
             <param name="can_interface">can0</param>
@@ -13,4 +13,21 @@
             <param name="speed_level">3</param>     <!-- 1/2/3 对应 30%/60%/100% -->
         </hardware>
+        <!-- ****************** 1号从臂的电机 ****************** -->
+        <joint name="s1__joint_motor_01">
+            <command_interface name="position" />
+            <state_interface name="position" />
+        </joint>
+        <joint name="s1__joint_motor_02">
+            <command_interface name="position" />
+            <state_interface name="position" />
+        </joint>
+        <joint name="s1__joint_motor_03">
+            <command_interface name="position" />
+            <state_interface name="position" />
+        </joint>
+        <joint name="s1__joint_motor_04">
+            <command_interface name="position" />
+            <state_interface name="position" />
+        </joint>
         <!-- ****************** 1号从臂的转动关节 ****************** -->
         <joint name="s1_j03_oc">
@@ -54,4 +71,21 @@
             <state_interface name="position" />
         </joint>
+        <!-- ****************** 1号从臂的电机 ****************** -->
+        <joint name="s2__joint_motor_01">
+            <command_interface name="position" />
+            <state_interface name="position" />
+        </joint>
+        <joint name="s2__joint_motor_02">
+            <command_interface name="position" />
+            <state_interface name="position" />
+        </joint>
+        <joint name="s2__joint_motor_03">
+            <command_interface name="position" />
+            <state_interface name="position" />
+        </joint>
+        <joint name="s2__joint_motor_04">
+            <command_interface name="position" />
+            <state_interface name="position" />
+        </joint>
         <!-- ****************** 2号从臂的转动关节 ****************** -->
         <joint name="s2_j03_oc">
@@ -96,7 +130,7 @@
         </joint>
     </ros2_control>
-    <ros2_control name="PSMCan1Hardware" type="system">
+    <ros2_control name="IntelligentCan1Ros2Control" type="system">
         <hardware>
-            <plugin>psm_can_hardware/PSMCan1HardwareInterface</plugin>
+            <plugin>psm_hardware_interface/IntelligentCan1HardwareInterface</plugin>
             <!-- CAN 通道 -->
             <param name="can_interface">can1</param>
@@ -107,4 +141,21 @@
             <param name="speed_level">3</param>     <!-- 1/2/3 对应 30%/60%/100% -->
         </hardware>
+        <!-- ****************** 3号从臂的电机 ****************** -->
+        <joint name="s3__joint_motor_01">
+            <command_interface name="position" />
+            <state_interface name="position" />
+        </joint>
+        <joint name="s3__joint_motor_02">
+            <command_interface name="position" />
+            <state_interface name="position" />
+        </joint>
+        <joint name="s3__joint_motor_03">
+            <command_interface name="position" />
+            <state_interface name="position" />
+        </joint>
+        <joint name="s3__joint_motor_04">
+            <command_interface name="position" />
+            <state_interface name="position" />
+        </joint>
         <!-- ****************** 3号从臂的转动关节 ****************** -->
         <joint name="s3_j03_oc">

Commit message: 蛇臂改好了，蛇头冲着-x了

File: src/leonardo_description/psm_description/10_snake/10_snake_links.xacro (robot description, xacro)
@@ -13,5 +13,5 @@
                     <mesh filename="${stl_path}/01.stl" scale="${mesh_scale}" />
                 </geometry>
-                <origin xyz="0 0 0" rpy="0 0 0" />
+                <origin xyz="0 0 0" rpy="0 0 ${pi/2}" />
                 <material name="${prefix}_link01" />
             </visual>
@@ -20,5 +20,5 @@
                     <mesh filename="${stl_path}/01.stl" scale="${mesh_scale}" />
                 </geometry>
-                <origin xyz="0 0 0" rpy="0 0 0" />
+                <origin xyz="0 0 0" rpy="0 0 ${pi/2}" />
             </collision>
             <xacro:snake_cylinder_inertia m="${link01_m}" r="${link01_r}" l="${link01_l}" o_xyz="0 0 0"
@@ -31,5 +31,5 @@
                     <mesh filename="${stl_path}/02.stl" scale="${mesh_scale}" />
                 </geometry>
-                <origin xyz="0 0 0" rpy="${pi} 0 0" />
+                <origin xyz="0 0 0" rpy="${pi} 0 ${pi/2}" />
                 <material name="${prefix}_link02" />
             </visual>
@@ -38,5 +38,5 @@
                     <mesh filename="${stl_path}/02.stl" scale="${mesh_scale}" />
                 </geometry>
-                <origin xyz="0 0 0" rpy="0 0 0" />
+                <origin xyz="0 0 0" rpy="0 0 ${pi/2}" />
             </collision>
             <xacro:snake_cylinder_inertia m="${link02_m}" r="${link02_r}" l="${link02_l}" o_xyz="0 0 0"
@@ -49,5 +49,5 @@
                     <mesh filename="${stl_path}/03.stl" scale="${mesh_scale}" />
                 </geometry>
-                <origin xyz="0 0 0" rpy="0 0 0" />
+                <origin xyz="0 0 0" rpy="0 0 ${pi/2}" />
                 <material name="${prefix}_link03" />
             </visual>
@@ -56,5 +56,5 @@
                     <mesh filename="${stl_path}/03.stl" scale="${mesh_scale}" />
                 </geometry>
-                <origin xyz="0 0 0" rpy="0 0 0" />
+                <origin xyz="0 0 0" rpy="0 0 ${pi/2}" />
             </collision>
             <xacro:snake_cylinder_inertia m="${link03_m}" r="${link03_r}" l="${link03_l}" o_xyz="0 0 0"
@@ -67,5 +67,5 @@
                     <mesh filename="${stl_path}/04.stl" scale="${mesh_scale}" />
                 </geometry>
-                <origin xyz="0 0 0" rpy="0 ${pi/2.0} 0" />
+                <origin xyz="0 0 0" rpy="0 ${pi/2.0} ${pi/2}" />
                 <material name="${prefix}_link04" />
             </visual>
@@ -74,5 +74,5 @@
                     <mesh filename="${stl_path}/04.stl" scale="${mesh_scale}" />
                 </geometry>
-                <origin xyz="0 0 0" rpy="0 0 0" />
+                <origin xyz="0 0 0" rpy="0 0 ${pi/2}" />
             </collision>
             <xacro:snake_cylinder_inertia m="${link04_m}" r="${link04_r}" l="${link04_l}" o_xyz="0 0 0"
@@ -85,5 +85,5 @@
                     <mesh filename="${stl_path}/05.stl" scale="${mesh_scale}" />
                 </geometry>
-                <origin xyz="0 0 0" rpy="0 0 0" />
+                <origin xyz="0 0 0" rpy="0 0 ${pi/2}" />
                 <material name="${prefix}_link05" />
             </visual>
@@ -92,5 +92,5 @@
                     <mesh filename="${stl_path}/05.stl" scale="${mesh_scale}" />
                 </geometry>
-                <origin xyz="0 0 0" rpy="0 0 0" />
+                <origin xyz="0 0 0" rpy="0 0 ${pi/2}" />
             </collision>
             <xacro:snake_cylinder_inertia m="${link05_m}" r="${link05_r}" l="${link05_l}" o_xyz="0 0 0"
@@ -103,5 +103,5 @@
                     <mesh filename="${stl_path}/06.stl" scale="${mesh_scale}" />
                 </geometry>
-                <origin xyz="0 0 0" rpy="0 0 0" />
+                <origin xyz="0 0 0" rpy="0 0 ${pi/2}" />
                 <material name="${prefix}_link06" />
             </visual>
@@ -110,5 +110,5 @@
                     <mesh filename="${stl_path}/06.stl" scale="${mesh_scale}" />
                 </geometry>
-                <origin xyz="0 0 0" rpy="0 0 0" />
+                <origin xyz="0 0 0" rpy="0 0 ${pi/2}" />
             </collision>
             <xacro:snake_cylinder_inertia m="${link06_m}" r="${link06_r}" l="${link06_l}" o_xyz="0 0 0"
@@ -121,5 +121,5 @@
                     <mesh filename="${stl_path}/07.stl" scale="${mesh_scale}" />
                 </geometry>
-                <origin xyz="0 0 0" rpy="${pi} 0 0" />
+                <origin xyz="0 0 0" rpy="${pi} 0 ${pi/2}" />
                 <material name="${prefix}_link07" />
             </visual>
@@ -128,5 +128,5 @@
                     <mesh filename="${stl_path}/07.stl" scale="${mesh_scale}" />
                 </geometry>
-                <origin xyz="0 0 0" rpy="0 0 0" />
+                <origin xyz="0 0 0" rpy="0 0 ${pi/2}" />
             </collision>
             <xacro:snake_cylinder_inertia m="${link07_m}" r="${link07_r}" l="${link07_l}" o_xyz="0 0 0"
@@ -139,5 +139,5 @@
                     <mesh filename="${stl_path}/08.stl" scale="${mesh_scale}" />
                 </geometry>
-                <origin xyz="0 0 0" rpy="${pi} ${pi/2.0} 0" />
+                <origin xyz="0 0 0" rpy="${pi} ${pi/2.0} ${pi/2}" />
                 <material name="${prefix}_link08" />
             </visual>
@@ -146,5 +146,5 @@
                     <mesh filename="${stl_path}/08.stl" scale="${mesh_scale}" />
                 </geometry>
-                <origin xyz="0 0 0" rpy="0 0 0" />
+                <origin xyz="0 0 0" rpy="0 0 ${pi/2}" />
             </collision>
             <xacro:snake_cylinder_inertia m="${link08_m}" r="${link08_r}" l="${link08_l}" o_xyz="0 0 0"
@@ -157,5 +157,5 @@
                     <mesh filename="${stl_path}/09.stl" scale="${mesh_scale}" />
                 </geometry>
-                <origin xyz="0 0 0" rpy="${pi} 0 0" />
+                <origin xyz="0 0 0" rpy="${pi} 0 ${pi/2}" />
                 <material name="${prefix}_link09" />
             </visual>
@@ -164,5 +164,5 @@
                     <mesh filename="${stl_path}/09.stl" scale="${mesh_scale}" />
                 </geometry>
-                <origin xyz="0 0 0" rpy="0 0 0" />
+                <origin xyz="0 0 0" rpy="0 0 ${pi/2}" />
             </collision>
             <xacro:snake_cylinder_inertia m="${link09_m}" r="${link09_r}" l="${link09_l}" o_xyz="0 0 0"
@@ -175,5 +175,5 @@
                     <mesh filename="${stl_path}/10.stl" scale="${mesh_scale}" />
                 </geometry>
-                <origin xyz="0 0 0" rpy="0 0 0" />
+                <origin xyz="0 0 0" rpy="0 0 ${pi/2}" />
                 <material name="${prefix}_link10" />
             </visual>
@@ -182,5 +182,5 @@
                     <mesh filename="${stl_path}/10.stl" scale="${mesh_scale}" />
                 </geometry>
-                <origin xyz="0 0 0" rpy="0 0 0" />
+                <origin xyz="0 0 0" rpy="0 0 ${pi/2}" />
             </collision>
             <xacro:snake_cylinder_inertia m="${link10_m}" r="${link10_r}" l="${link10_l}" o_xyz="0 0 0"
@@ -193,5 +193,5 @@
                     <mesh filename="${stl_path}/11.stl" scale="${mesh_scale}" />
                 </geometry>
-                <origin xyz="0 0 0" rpy="0 0 0" />
+                <origin xyz="0 0 0" rpy="0 0 ${pi/2}" />
                 <material name="${prefix}_link11" />
             </visual>
@@ -200,5 +200,5 @@
                     <mesh filename="${stl_path}/11.stl" scale="${mesh_scale}" />
                 </geometry>
-                <origin xyz="0 0 0" rpy="0 0 0" />
+                <origin xyz="0 0 0" rpy="0 0 ${pi/2}" />
             </collision>
             <xacro:snake_cylinder_inertia m="${link11_m}" r="${link11_r}" l="${link11_l}" o_xyz="0 0 0"
@@ -211,5 +211,5 @@
                     <mesh filename="${stl_path}/12.stl" scale="${mesh_scale}" />
                 </geometry>
-                <origin xyz="0 0 0" rpy="0 ${pi/2.0} 0" />
+                <origin xyz="0 0 0" rpy="0 ${pi/2.0} ${pi/2}" />
                 <material name="${prefix}_link12" />
             </visual>
@@ -218,5 +218,5 @@
                     <mesh filename="${stl_path}/12.stl" scale="${mesh_scale}" />
                 </geometry>
-                <origin xyz="0 0 0" rpy="0 0 0" />
+                <origin xyz="0 0 0" rpy="0 0 ${pi/2}" />
             </collision>
             <xacro:snake_cylinder_inertia m="${link12_m}" r="${link12_r}" l="${link12_l}" o_xyz="0 0 0"
@@ -229,5 +229,5 @@
                     <mesh filename="${stl_path}/13.stl" scale="${mesh_scale}" />
                 </geometry>
-                <origin xyz="0 0 0" rpy="0 0 0" />
+                <origin xyz="0 0 0" rpy="0 0 ${pi/2}" />
                 <material name="${prefix}_link13" />
             </visual>
@@ -236,5 +236,5 @@
                     <mesh filename="${stl_path}/13.stl" scale="${mesh_scale}" />
                 </geometry>
-                <origin xyz="0 0 0" rpy="0 0 0" />
+                <origin xyz="0 0 0" rpy="0 0 ${pi/2}" />
             </collision>
             <xacro:snake_cylinder_inertia m="${link13_m}" r="${link13_r}" l="${link13_l}" o_xyz="0 0 0"
@@ -247,5 +247,5 @@
                     <mesh filename="${stl_path}/14.stl" scale="${mesh_scale}" />
                 </geometry>
-                <origin xyz="0 0 0" rpy="0 ${pi/2.0} 0" />
+                <origin xyz="0 0 0" rpy="0 ${pi/2.0} ${pi/2}" />
                 <material name="${prefix}_link14" />
             </visual>
@@ -254,5 +254,5 @@
                     <mesh filename="${stl_path}/14.stl" scale="${mesh_scale}" />
                 </geometry>
-                <origin xyz="0 0 0" rpy="0 0 0" />
+                <origin xyz="0 0 0" rpy="0 0 ${pi/2}" />
             </collision>
             <xacro:snake_cylinder_inertia m="${link14_m}" r="${link14_r}" l="${link14_l}" o_xyz="0 0 0"
@@ -265,5 +265,5 @@
                     <mesh filename="${stl_path}/15.stl" scale="${mesh_scale}" />
                 </geometry>
-                <origin xyz="0 0 0" rpy="0 0 0" />
+                <origin xyz="0 0 0" rpy="0 0 ${pi/2}" />
                 <material name="${prefix}_link15" />
             </visual>
@@ -272,5 +272,5 @@
                     <mesh filename="${stl_path}/15.stl" scale="${mesh_scale}" />
                 </geometry>
-                <origin xyz="0 0 0" rpy="0 0 0" />
+                <origin xyz="0 0 0" rpy="0 0 ${pi/2}" />
             </collision>
             <xacro:snake_cylinder_inertia m="${link15_m}" r="${link15_r}" l="${link15_l}" o_xyz="0 0 0"
@@ -283,5 +283,5 @@
                     <mesh filename="${stl_path}/16.stl" scale="${mesh_scale}" />
                 </geometry>
-                <origin xyz="0 0 0" rpy="0 0 0" />
+                <origin xyz="0 0 0" rpy="0 0 ${pi/2}" />
                 <material name="${prefix}_link16" />
             </visual>
@@ -290,5 +290,5 @@
                     <mesh filename="${stl_path}/16.stl" scale="${mesh_scale}" />
                 </geometry>
-                <origin xyz="0 0 0" rpy="0 0 0" />
+                <origin xyz="0 0 0" rpy="0 0 ${pi/2}" />
             </collision>
             <xacro:snake_cylinder_inertia m="${link16_m}" r="${link16_r}" l="${link16_l}" o_xyz="0 0 0"
@@ -301,5 +301,5 @@
                     <mesh filename="${stl_path}/17.stl" scale="${mesh_scale}" />
                 </geometry>
-                <origin xyz="0 0 0" rpy="0 0 ${pi/2}" />
+                <origin xyz="0 0 0" rpy="0 0 ${pi}" />
                 <material name="${prefix}_link17" />
             </visual>
@@ -308,5 +308,5 @@
                     <mesh filename="${stl_path}/17.stl" scale="${mesh_scale}" />
                 </geometry>
-                <origin xyz="0 0 0" rpy="0 0 0" />
+                <origin xyz="0 0 0" rpy="0 0 ${pi/2}" />
             </collision>
             <xacro:snake_cylinder_inertia m="${link17_m}" r="${link17_r}" l="${link17_l}" o_xyz="0 0 0"
@@ -319,5 +319,5 @@
                     <mesh filename="${stl_path}/18.stl" scale="${mesh_scale}" />
                 </geometry>
-                <origin xyz="0 0 0" rpy="0 0 ${pi}" />
+                <origin xyz="0 0 0" rpy="0 0 ${pi * 1.5}" />
                 <material name="${prefix}_link18" />
             </visual>
@@ -326,5 +326,5 @@
                     <mesh filename="${stl_path}/18.stl" scale="${mesh_scale}" />
                 </geometry>
-                <origin xyz="0 0 0" rpy="0 0 0" />
+                <origin xyz="0 0 0" rpy="0 0 ${pi/2}" />
             </collision>
             <xacro:snake_cylinder_inertia m="${link18_m}" r="${link18_r}" l="${link18_l}" o_xyz="0 0 0"
@@ -337,5 +337,5 @@
                     <mesh filename="${stl_path}/19.stl" scale="${mesh_scale}" />
                 </geometry>
-                <origin xyz="0 0 0" rpy="${pi/2.0} 0 0" />
+                <origin xyz="0 0 0" rpy="${pi/2.0} 0 ${pi/2}" />
                 <material name="${prefix}_link19" />
             </visual>
@@ -344,5 +344,5 @@
                     <mesh filename="${stl_path}/19.stl" scale="${mesh_scale}" />
                 </geometry>
-                <origin xyz="0 0 0" rpy="0 0 0" />
+                <origin xyz="0 0 0" rpy="0 0 ${pi/2}" />
             </collision>
             <xacro:snake_cylinder_inertia m="${link19_m}" r="${link19_r}" l="${link19_l}" o_xyz="0 0 0"
@@ -355,5 +355,5 @@
                     <mesh filename="${stl_path}/20.stl" scale="${mesh_scale}" />
                 </geometry>
-                <origin xyz="0 0 -0.004" rpy="${pi/2.0} 0 0" />
+                <origin xyz="0 0 -0.004" rpy="${pi/2.0} 0 ${pi/2}" />
                 <material name="${prefix}_link20" />
             </visual>
@@ -362,5 +362,5 @@
                     <mesh filename="${stl_path}/20.stl" scale="${mesh_scale}" />
                 </geometry>
-                <origin xyz="0 0 0" rpy="0 0 0" />
+                <origin xyz="0 0 0" rpy="0 0 ${pi/2}" />
             </collision>
             <xacro:snake_cylinder_inertia m="${link20_m}" r="${link20_r}" l="${link20_l}" o_xyz="0 0 0"
@@ -373,5 +373,5 @@
                     <mesh filename="${stl_path}/21.stl" scale="${mesh_scale}" />
                 </geometry>
-                <origin xyz="0 0 0" rpy="${pi/2.0} 0 0" />
+                <origin xyz="0 0 0" rpy="${pi/2.0} 0 ${pi/2}" />
                 <material name="${prefix}_link21" />
             </visual>
@@ -380,5 +380,5 @@
                     <mesh filename="${stl_path}/21.stl" scale="${mesh_scale}" />
                 </geometry>
-                <origin xyz="0 0 0" rpy="0 0 0" />
+                <origin xyz="0 0 0" rpy="0 0 ${pi/2}" />
             </collision>
             <xacro:snake_cylinder_inertia m="${link21_m}" r="${link21_r}" l="${link21_l}" o_xyz="0 0 0"
@@ -391,5 +391,5 @@
                     <mesh filename="${stl_path}/22.stl" scale="${mesh_scale}" />
                 </geometry>
-                <origin xyz="0 0 0" rpy="${pi/2.0} ${pi} 0" />
+                <origin xyz="0 0 0" rpy="${pi/2.0} ${pi} ${pi/2}" />
                 <material name="${prefix}_link22" />
             </visual>
@@ -398,5 +398,5 @@
                     <mesh filename="${stl_path}/22.stl" scale="${mesh_scale}" />
                 </geometry>
-                <origin xyz="0 0 0" rpy="0 0 0" />
+                <origin xyz="0 0 0" rpy="0 0 ${pi/2}" />
             </collision>
             <xacro:snake_cylinder_inertia m="${link22_m}" r="${link22_r}" l="${link22_l}" o_xyz="0 0 0"
