Commit message: 蛇臂改好了，蛇头冲着-x了

File: src/leonardo_description/psm_description/10_snake/11_snake_joints.xacro (robot description, xacro)
@@ -1,6 +1,5 @@
 <?xml version="1.0" encoding="UTF-8"?>
-<!-- 蛇形机械臂关节定义：适配 22 个 link，统一关节命名 -->
 <robot xmlns:xacro="http://www.ros.org/wiki/xacro">
-    <!-- ==========  y轴偏移量  ========== -->
+    <!-- ==========  偏移量  ========== -->
     <xacro:property name="y_offset_01_02" value="0.0514" />
     <xacro:property name="y_offset_02_03" value="0.0013" />
@@ -12,9 +11,9 @@
     <xacro:property name="y_offset_16_17" value="0.01172" />
     <xacro:property name="y_offset_17_18" value="0.00728" />
-    <xacro:property name="y_offset_18_19" value="-0.0013" />
+    <xacro:property name="y_offset_18_19" value="-0.0013" /> <!-- 注意：这个是负数 -->
     <xacro:property name="y_offset_19_20" value="0.005" />
     <xacro:property name="y_offset_20_21" value="0.0" />
     <xacro:property name="y_offset_20_22" value="0.0" />
-    <!-- 蛇骨公转半径：两齿轮中心距（两齿轮半径之和） -->
+    <!-- 蛇骨公转半径 -->
     <xacro:property name="orbit_r" value="0.0025" />
     <!-- 蛇骨公转角度限位（±22.5°） -->
@@ -44,5 +43,5 @@
     <!-- ========== 宏定义：生成所有关节 ========== -->
     <xacro:macro name="get_snake_joints" params="prefix">
-        <!-- ****************************************  4个虚拟旋转joint  **************************************** -->
+        <!-- 4个虚拟旋转joint -->
         <joint name="${prefix}_joint_motor_01" type="revolute">
             <parent link="${prefix}_01" />
@@ -55,5 +54,5 @@
             <parent link="${prefix}_01" />
             <child link="${prefix}_link_for_motor_02" />
-            <origin xyz="0.005 0 0.01" rpy="0 0 0" />
+            <origin xyz="0 0.005 0.01" rpy="0 0 0" />
             <axis xyz="0 0 1" />
             <limit effort="${effort}" velocity="${velocity}" lower="${-pi/2.0}" upper="${pi/2.0}" />
@@ -62,5 +61,5 @@
             <parent link="${prefix}_01" />
             <child link="${prefix}_link_for_motor_03" />
-            <origin xyz="0.01 0 0.01" rpy="0 0 0" />
+            <origin xyz="0 0.01 0.01" rpy="0 0 0" />
             <axis xyz="0 0 1" />
             <limit effort="${effort}" velocity="${velocity}" lower="${-pi/2.0}" upper="${pi/2.0}" />
@@ -69,49 +68,44 @@
             <parent link="${prefix}_01" />
             <child link="${prefix}_link_for_motor_04" />
-            <origin xyz="0.015 0 0.01" rpy="0 0 0" />
-            <axis xyz="0 0 1" />
-            <limit effort="${effort}" velocity="${velocity}" lower="${-pi/2.0}" upper="${pi/2.0}" />
-        </joint>
-        <!-- ****************************************  link01 -> link02  **************************************** -->
+            <origin xyz="0 0.015 0.01" rpy="0 0 0" />
+            <axis xyz="0 0 1" />
+            <limit effort="${effort}" velocity="${velocity}" lower="${-pi/2.0}" upper="${pi/2.0}" />
+        </joint>
+        <!-- link01 -> link02 -->
         <joint name="${prefix}_joint_01_02" type="fixed">
             <parent link="${prefix}_01" />
             <child link="${prefix}_02" />
-            <origin xyz="0 ${y_offset_01_02} 0" rpy="0 0 0" />
-        </joint>
-        <!-- ****************************************  link02 -> link03  **************************************** -->
+            <origin xyz="-${y_offset_01_02} 0 0" rpy="0 0 0" />
+        </joint>
+        <!-- link02 -> link03 -->
         <joint name="${prefix}_joint_02_03" type="fixed">
             <parent link="${prefix}_02" />
             <child link="${prefix}_03" />
-            <origin xyz="0 ${y_offset_02_03} 0" rpy="0 0 0" />
-        </joint>
-        <!-- ****************************************  link03 -> link04  **************************************** -->
+            <origin xyz="-${y_offset_02_03} 0 0" rpy="0 0 0" />
+        </joint>
+        <!-- link03 -> link04 -->
         <link name="${prefix}_orbit_carrier_03" />
         <link name="${prefix}_gear_center_04" />
-        <!-- 公转关节：link03 -> 公转载体 -->
         <joint name="${prefix}_j03_oc" type="revolute">
             <parent link="${prefix}_03" />
             <child link="${prefix}_orbit_carrier_03" />
-            <origin xyz="0 ${origin_gear_center_03_L} 0" rpy="0 0 0" />
-            <axis xyz="0 0 1" />
-            <limit effort="${effort}" velocity="${velocity}"
-                lower="${orbit_lower}" upper="${orbit_upper}" />
-        </joint>
-        <!-- 自转关节：公转载体 -> link04 齿轮中心 -->
-        <!-- 公转半径 orbit_r；mimic 公转 1:1 实现自转 -->
+            <origin xyz="-${origin_gear_center_03_L} 0 0" rpy="0 0 0" />
+            <axis xyz="0 0 1" />
+            <limit effort="${effort}" velocity="${velocity}" lower="${orbit_lower}" upper="${orbit_upper}" />
+        </joint>
         <joint name="${prefix}_joint_04_spin" type="continuous">
             <parent link="${prefix}_orbit_carrier_03" />
             <child link="${prefix}_gear_center_04" />
-            <origin xyz="0 ${orbit_r} 0" rpy="0 0 0" />
+            <origin xyz="-${orbit_r} 0 0" rpy="0 0 0" />
             <axis xyz="0 0 1" />
             <limit effort="${effort}" velocity="${velocity}" />
             <mimic joint="${prefix}_j03_oc" multiplier="1" offset="0" />
         </joint>
-        <!-- 固定关节：link04 齿轮中心 -> link04 原点 -->
         <joint name="${prefix}_joint_04_mount" type="fixed">
             <parent link="${prefix}_gear_center_04" />
             <child link="${prefix}_04" />
-            <origin xyz="0 ${origin_gear_center_04_R} 0" rpy="0 0 0" />
-        </joint>
-        <!-- ****************************************  link04 -> link05  **************************************** -->
+            <origin xyz="-${origin_gear_center_04_R} 0 0" rpy="0 0 0" />
+        </joint>
+        <!-- link04 -> link05 -->
         <link name="${prefix}_orbit_carrier_04" />
         <link name="${prefix}_gear_center_05" />
@@ -119,6 +113,6 @@
             <parent link="${prefix}_04" />
             <child link="${prefix}_orbit_carrier_04" />
-            <origin xyz="0 ${origin_gear_center_04_L} 0" rpy="0 0 0" />
-            <axis xyz="1 0 0" />
+            <origin xyz="-${origin_gear_center_04_L} 0 0" rpy="0 0 0" />
+            <axis xyz="0 1 0" />
             <limit effort="${effort}" velocity="${velocity}" lower="${orbit_lower}" upper="${orbit_upper}" />
         </joint>
@@ -126,6 +120,6 @@
             <parent link="${prefix}_orbit_carrier_04" />
             <child link="${prefix}_gear_center_05" />
-            <origin xyz="0 ${orbit_r} 0" rpy="0 0 0" />
-            <axis xyz="1 0 0" />
+            <origin xyz="-${orbit_r} 0 0" rpy="0 0 0" />
+            <axis xyz="0 1 0" />
             <limit effort="${effort}" velocity="${velocity}" />
             <mimic joint="${prefix}_j04_oc" multiplier="1" offset="0" />
@@ -134,19 +128,19 @@
             <parent link="${prefix}_gear_center_05" />
             <child link="${prefix}_05" />
-            <origin xyz="0 ${origin_gear_center_05_R} 0" rpy="0 0 0" />
-        </joint>
-        <!-- ****************************************  link05 -> link06  **************************************** -->
+            <origin xyz="-${origin_gear_center_05_R} 0 0" rpy="0 0 0" />
+        </joint>
+        <!-- link05 -> link06 -->
         <joint name="${prefix}_joint_05_06" type="fixed">
             <parent link="${prefix}_05" />
             <child link="${prefix}_06" />
-            <origin xyz="0 ${y_offset_05_06} 0" rpy="0 0 0" />
-        </joint>
-        <!-- ****************************************  link06 -> link07  **************************************** -->
+            <origin xyz="-${y_offset_05_06} 0 0" rpy="0 0 0" />
+        </joint>
+        <!-- link06 -> link07 -->
         <joint name="${prefix}_joint_06_07" type="fixed">
             <parent link="${prefix}_06" />
             <child link="${prefix}_07" />
-            <origin xyz="0 ${y_offset_06_07} 0" rpy="0 0 0" />
-        </joint>
-        <!-- ****************************************  link07 -> link08  **************************************** -->
+            <origin xyz="-${y_offset_06_07} 0 0" rpy="0 0 0" />
+        </joint>
+        <!-- link07 -> link08 -->
         <link name="${prefix}_orbit_carrier_07" />
         <link name="${prefix}_gear_center_08" />
@@ -154,6 +148,6 @@
             <parent link="${prefix}_07" />
             <child link="${prefix}_orbit_carrier_07" />
-            <origin xyz="0 ${origin_gear_center_07_L} 0" rpy="0 0 0" />
-            <axis xyz="1 0 0" />
+            <origin xyz="-${origin_gear_center_07_L} 0 0" rpy="0 0 0" />
+            <axis xyz="0 1 0" />
             <limit effort="${effort}" velocity="${velocity}" lower="${orbit_lower}" upper="${orbit_upper}" />
         </joint>
@@ -161,6 +155,6 @@
             <parent link="${prefix}_orbit_carrier_07" />
             <child link="${prefix}_gear_center_08" />
-            <origin xyz="0 ${orbit_r} 0" rpy="0 0 0" />
-            <axis xyz="1 0 0" />
+            <origin xyz="-${orbit_r} 0 0" rpy="0 0 0" />
+            <axis xyz="0 1 0" />
             <limit effort="${effort}" velocity="${velocity}" />
             <mimic joint="${prefix}_j07_oc" multiplier="1" offset="0" />
@@ -169,7 +163,7 @@
             <parent link="${prefix}_gear_center_08" />
             <child link="${prefix}_08" />
-            <origin xyz="0 ${origin_gear_center_08_R} 0" rpy="0 0 0" />
-        </joint>
-        <!-- ****************************************  link08 -> link09  **************************************** -->
+            <origin xyz="-${origin_gear_center_08_R} 0 0" rpy="0 0 0" />
+        </joint>
+        <!-- link08 -> link09 -->
         <link name="${prefix}_orbit_carrier_08" />
         <link name="${prefix}_gear_center_09" />
@@ -177,5 +171,5 @@
             <parent link="${prefix}_08" />
             <child link="${prefix}_orbit_carrier_08" />
-            <origin xyz="0 ${origin_gear_center_08_L} 0" rpy="0 0 0" />
+            <origin xyz="-${origin_gear_center_08_L} 0 0" rpy="0 0 0" />
             <axis xyz="0 0 1" />
             <limit effort="${effort}" velocity="${velocity}" lower="${orbit_lower}" upper="${orbit_upper}" />
@@ -184,5 +178,5 @@
             <parent link="${prefix}_orbit_carrier_08" />
             <child link="${prefix}_gear_center_09" />
-            <origin xyz="0 ${orbit_r} 0" rpy="0 0 0" />
+            <origin xyz="-${orbit_r} 0 0" rpy="0 0 0" />
             <axis xyz="0 0 1" />
             <limit effort="${effort}" velocity="${velocity}" />
@@ -192,19 +186,19 @@
             <parent link="${prefix}_gear_center_09" />
             <child link="${prefix}_09" />
-            <origin xyz="0 ${origin_gear_center_09_R} 0" rpy="0 0 0" />
-        </joint>
-        <!-- ****************************************  link09 -> link10  **************************************** -->
+            <origin xyz="-${origin_gear_center_09_R} 0 0" rpy="0 0 0" />
+        </joint>
+        <!-- link09 -> link10 -->
         <joint name="${prefix}_joint_09_10" type="fixed">
             <parent link="${prefix}_09" />
             <child link="${prefix}_10" />
-            <origin xyz="0 ${y_offset_09_10} 0" rpy="0 0 0" />
-        </joint>
-        <!-- ****************************************  link10 -> link11  **************************************** -->
+            <origin xyz="-${y_offset_09_10} 0 0" rpy="0 0 0" />
+        </joint>
+        <!-- link10 -> link11 -->
         <joint name="${prefix}_joint_10_11" type="fixed">
             <parent link="${prefix}_10" />
             <child link="${prefix}_11" />
-            <origin xyz="0 ${y_offset_10_11} 0" rpy="0 0 0" />
-        </joint>
-        <!-- ****************************************  link11 -> link12  **************************************** -->
+            <origin xyz="-${y_offset_10_11} 0 0" rpy="0 0 0" />
+        </joint>
+        <!-- link11 -> link12 -->
         <link name="${prefix}_orbit_carrier_11" />
         <link name="${prefix}_gear_center_12" />
@@ -212,5 +206,5 @@
             <parent link="${prefix}_11" />
             <child link="${prefix}_orbit_carrier_11" />
-            <origin xyz="0 ${origin_gear_center_11_L} 0" rpy="0 0 0" />
+            <origin xyz="-${origin_gear_center_11_L} 0 0" rpy="0 0 0" />
             <axis xyz="0 0 1" />
             <limit effort="${effort}" velocity="${velocity}" lower="${orbit_lower}" upper="${orbit_upper}" />
@@ -219,5 +213,5 @@
             <parent link="${prefix}_orbit_carrier_11" />
             <child link="${prefix}_gear_center_12" />
-            <origin xyz="0 ${orbit_r} 0" rpy="0 0 0" />
+            <origin xyz="-${orbit_r} 0 0" rpy="0 0 0" />
             <axis xyz="0 0 1" />
             <limit effort="${effort}" velocity="${velocity}" />
@@ -227,7 +221,7 @@
             <parent link="${prefix}_gear_center_12" />
             <child link="${prefix}_12" />
-            <origin xyz="0 ${origin_gear_center_12_R} 0" rpy="0 0 0" />
-        </joint>
-        <!-- ****************************************  link12 -> link13  **************************************** -->
+            <origin xyz="-${origin_gear_center_12_R} 0 0" rpy="0 0 0" />
+        </joint>
+        <!-- link12 -> link13 -->
         <link name="${prefix}_orbit_carrier_12" />
         <link name="${prefix}_gear_center_13" />
@@ -235,6 +229,6 @@
             <parent link="${prefix}_12" />
             <child link="${prefix}_orbit_carrier_12" />
-            <origin xyz="0 ${origin_gear_center_12_L} 0" rpy="0 0 0" />
-            <axis xyz="1 0 0" />
+            <origin xyz="-${origin_gear_center_12_L} 0 0" rpy="0 0 0" />
+            <axis xyz="0 1 0" />
             <limit effort="${effort}" velocity="${velocity}" lower="${orbit_lower}" upper="${orbit_upper}" />
         </joint>
@@ -242,6 +236,6 @@
             <parent link="${prefix}_orbit_carrier_12" />
             <child link="${prefix}_gear_center_13" />
-            <origin xyz="0 ${orbit_r} 0" rpy="0 0 0" />
-            <axis xyz="1 0 0" />
+            <origin xyz="-${orbit_r} 0 0" rpy="0 0 0" />
+            <axis xyz="0 1 0" />
             <limit effort="${effort}" velocity="${velocity}" />
             <mimic joint="${prefix}_j12_oc" multiplier="1" offset="0" />
@@ -250,7 +244,7 @@
             <parent link="${prefix}_gear_center_13" />
             <child link="${prefix}_13" />
-            <origin xyz="0 ${origin_gear_center_13_R} 0" rpy="0 0 0" />
-        </joint>
-        <!-- ****************************************  link13 -> link14  **************************************** -->
+            <origin xyz="-${origin_gear_center_13_R} 0 0" rpy="0 0 0" />
+        </joint>
+        <!-- link13 -> link14 -->
         <link name="${prefix}_orbit_carrier_13" />
         <link name="${prefix}_gear_center_14" />
@@ -258,5 +252,5 @@
             <parent link="${prefix}_13" />
             <child link="${prefix}_orbit_carrier_13" />
-            <origin xyz="0 ${origin_gear_center_13_L} 0" rpy="0 0 0" />
+            <origin xyz="-${origin_gear_center_13_L} 0 0" rpy="0 0 0" />
             <axis xyz="0 0 1" />
             <limit effort="${effort}" velocity="${velocity}" lower="${orbit_lower}" upper="${orbit_upper}" />
@@ -265,5 +259,5 @@
             <parent link="${prefix}_orbit_carrier_13" />
             <child link="${prefix}_gear_center_14" />
-            <origin xyz="0 ${orbit_r} 0" rpy="0 0 0" />
+            <origin xyz="-${orbit_r} 0 0" rpy="0 0 0" />
             <axis xyz="0 0 1" />
             <limit effort="${effort}" velocity="${velocity}" />
@@ -273,7 +267,7 @@
             <parent link="${prefix}_gear_center_14" />
             <child link="${prefix}_14" />
-            <origin xyz="0 ${origin_gear_center_14_R} 0" rpy="0 0 0" />
-        </joint>
-        <!-- ****************************************  link14 -> link15  **************************************** -->
+            <origin xyz="-${origin_gear_center_14_R} 0 0" rpy="0 0 0" />
+        </joint>
+        <!-- link14 -> link15 -->
         <link name="${prefix}_orbit_carrier_14" />
         <link name="${prefix}_gear_center_15" />
@@ -281,6 +275,6 @@
             <parent link="${prefix}_14" />
             <child link="${prefix}_orbit_carrier_14" />
-            <origin xyz="0 ${origin_gear_center_14_L} 0" rpy="0 0 0" />
-            <axis xyz="1 0 0" />
+            <origin xyz="-${origin_gear_center_14_L} 0 0" rpy="0 0 0" />
+            <axis xyz="0 1 0" />
             <limit effort="${effort}" velocity="${velocity}" lower="${orbit_lower}" upper="${orbit_upper}" />
         </joint>
@@ -288,6 +282,6 @@
             <parent link="${prefix}_orbit_carrier_14" />
             <child link="${prefix}_gear_center_15" />
-            <origin xyz="0 ${orbit_r} 0" rpy="0 0 0" />
-            <axis xyz="1 0 0" />
+            <origin xyz="-${orbit_r} 0 0" rpy="0 0 0" />
+            <axis xyz="0 1 0" />
             <limit effort="${effort}" velocity="${velocity}" />
             <mimic joint="${prefix}_j14_oc" multiplier="1" offset="0" />
@@ -296,51 +290,52 @@
             <parent link="${prefix}_gear_center_15" />
             <child link="${prefix}_15" />
-            <origin xyz="0 ${origin_gear_center_15_R} 0" rpy="0 0 0" />
-        </joint>
-        <!-- ****************************************  link15 -> link16  **************************************** -->
+            <origin xyz="-${origin_gear_center_15_R} 0 0" rpy="0 0 0" />
+        </joint>
+        <!-- link15 -> link16 -->
         <joint name="${prefix}_joint_15_16" type="fixed">
             <parent link="${prefix}_15" />
             <child link="${prefix}_16" />
-            <origin xyz="0 ${y_offset_15_16} 0" rpy="0 0 0" />
-        </joint>
-        <!-- ****************************************  link16 -> link17  **************************************** -->
+            <origin xyz="-${y_offset_15_16} 0 0" rpy="0 0 0" />
+        </joint>
+        <!-- link16 -> link17 -->
         <joint name="${prefix}_joint_16_17" type="fixed">
             <parent link="${prefix}_16" />
             <child link="${prefix}_17" />
-            <origin xyz="0 ${y_offset_16_17} 0" rpy="0 0 0" />
-        </joint>
-        <!-- ****************************************  link17 -> link18  **************************************** -->
+            <origin xyz="-${y_offset_16_17} 0 0" rpy="0 0 0" />
+        </joint>
+        <!-- link17 -> link18 -->
         <joint name="${prefix}_j17_18" type="revolute">
             <parent link="${prefix}_17" />
             <child link="${prefix}_18" />
-            <origin xyz="0 ${y_offset_17_18} 0" rpy="0 0 0" />
-            <axis xyz="0 1 0" />
-            <limit effort="${effort}" velocity="${velocity}" lower="${-pi/2.0}" upper="${pi/2.0}" />
-        </joint>
-        <!-- ****************************************  link18 -> link19  **************************************** -->
+            <origin xyz="-${y_offset_17_18} 0 0" rpy="0 0 0" />
+            <axis xyz="-1 0 0" />
+            <limit effort="${effort}" velocity="${velocity}" lower="${-pi/2.0}" upper="${pi/2.0}" />
+        </joint>
+        <!-- link18 -> link19 -->
         <joint name="${prefix}_joint_18_19" type="fixed">
             <parent link="${prefix}_18" />
             <child link="${prefix}_19" />
-            <origin xyz="0 ${y_offset_18_19} 0" rpy="0 0 0" />
-        </joint>
-        <!-- ****************************************  link19 -> link20  **************************************** -->
+            <!-- 核心修复：改为 ${-y_offset_18_19}，防止出现双负号 -->
+            <origin xyz="${-y_offset_18_19} 0 0" rpy="0 0 0" />
+        </joint>
+        <!-- link19 -> link20 -->
         <joint name="${prefix}_joint_19_20" type="fixed">
             <parent link="${prefix}_19" />
             <child link="${prefix}_20" />
-            <origin xyz="0 ${y_offset_19_20} 0" rpy="0 0 0" />
-        </joint>
-        <!-- link20 -> link21 （主动钳） -->
+            <origin xyz="-${y_offset_19_20} 0 0" rpy="0 0 0" />
+        </joint>
+        <!-- link20 -> link21 -->
         <joint name="${prefix}_j20_21" type="revolute">
             <parent link="${prefix}_20" />
             <child link="${prefix}_21" />
-            <origin xyz="0 ${y_offset_20_21} 0" rpy="0 0 0" />
+            <origin xyz="-${y_offset_20_21} 0 0" rpy="0 0 0" />
             <axis xyz="0 0 1" />
             <limit effort="${effort}" velocity="${velocity}" lower="0" upper="${pi/6.0}" />
         </joint>
-        <!-- link20 -> link22 （镜像钳） -->
+        <!-- link20 -> link22 -->
         <joint name="${prefix}_joint_20_22" type="revolute">
             <parent link="${prefix}_20" />
             <child link="${prefix}_22" />
-            <origin xyz="0 ${y_offset_20_22} 0" rpy="0 0 0" />
+            <origin xyz="-${y_offset_20_22} 0 0" rpy="0 0 0" />
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
File: src/leonardo_description/psm_description/10_snake/69_snake_robot.xacro (robot description, xacro)
@@ -24,9 +24,14 @@
     <!-- 17 生成 base_footprint_snake 固定基座 -->
     <link name="base_footprint_snake" />
+    <!--
+        蛇头朝向 -X，轴线沿 X。
+        原本的横向排布（X轴 0.05, 0.1 的偏移）映射到 Y 轴上。
+    -->
     <joint name="s1_j01_base" type="prismatic">
         <parent link="base_footprint_snake" />
         <child link="s1_01" />
         <origin xyz="0 0 0" rpy="0 0 0" />
-        <axis xyz="0 1 0" />
+        <!-- 沿 -X 轴平移（朝向蛇头方向） -->
+        <axis xyz="-1 0 0" />
         <limit effort="10.0" velocity="0.5" lower="-0.1" upper="0.1" />
     </joint>
@@ -34,6 +39,7 @@
         <parent link="base_footprint_snake" />
         <child link="s2_01" />
-        <origin xyz="0.05 0 0" rpy="0 0 0" />
-        <axis xyz="0 1 0" />
+        <!-- Y 轴方向拉开 0.05 米 -->
+        <origin xyz="0 0.05 0" rpy="0 0 0" />
+        <axis xyz="-1 0 0" />
         <limit effort="10.0" velocity="0.5" lower="-0.1" upper="0.1" />
     </joint>
@@ -41,6 +47,7 @@
         <parent link="base_footprint_snake" />
         <child link="s3_01" />
-        <origin xyz="0.1 0 0" rpy="0 0 0" />
-        <axis xyz="0 1 0" />
+        <!-- Y 轴方向拉开 0.1 米 -->
+        <origin xyz="0 0.1 0" rpy="0 0 0" />
+        <axis xyz="-1 0 0" />
         <limit effort="10.0" velocity="0.5" lower="-0.1" upper="0.1" />
     </joint>
