Commit message: psm从臂改成6电机，还有1个直线电机是前后运动

File: src/leonardo_description/psm_description/10_snake/10_snake_links.xacro (robot description, xacro)
@@ -7,4 +7,6 @@
         <link name="${prefix}_link_for_motor_03" />
         <link name="${prefix}_link_for_motor_04" />
+        <link name="${prefix}_link_for_motor_05" />
+        <link name="${prefix}_link_for_motor_06" />
         <!-- ==================== Link 01 ==================== -->
         <link name="${prefix}_01">

File: src/leonardo_description/psm_description/10_snake/11_snake_joints.xacro (robot description, xacro)
@@ -43,5 +43,5 @@
     <!-- ========== 宏定义：生成所有关节 ========== -->
     <xacro:macro name="get_snake_joints" params="prefix">
-        <!-- 4个虚拟旋转joint -->
+        <!-- 6个虚拟旋转joint -->
         <joint name="${prefix}_joint_motor_01" type="revolute">
             <parent link="${prefix}_01" />
@@ -69,4 +69,18 @@
             <child link="${prefix}_link_for_motor_04" />
             <origin xyz="0 0.015 0.01" rpy="0 0 0" />
+            <axis xyz="0 0 1" />
+            <limit effort="${effort}" velocity="${velocity}" lower="${-pi/2.0}" upper="${pi/2.0}" />
+        </joint>
+        <joint name="${prefix}_joint_motor_05" type="revolute">
+            <parent link="${prefix}_01" />
+            <child link="${prefix}_link_for_motor_05" />
+            <origin xyz="0 0.02 0.01" rpy="0 0 0" />
+            <axis xyz="0 0 1" />
+            <limit effort="${effort}" velocity="${velocity}" lower="${-pi/2.0}" upper="${pi/2.0}" />
+        </joint>
+        <joint name="${prefix}_joint_motor_06" type="revolute">
+            <parent link="${prefix}_01" />
+            <child link="${prefix}_link_for_motor_06" />
+            <origin xyz="0 0.025 0.01" rpy="0 0 0" />
             <axis xyz="0 0 1" />
             <limit effort="${effort}" velocity="${velocity}" lower="${-pi/2.0}" upper="${pi/2.0}" />

File: src/leonardo_description/psm_description/10_snake/88_snake_robot.ros2_control.xacro (robot description, xacro)
@@ -30,4 +30,12 @@
             <state_interface name="position" />
         </joint>
+        <joint name="s1_joint_motor_05">
+            <command_interface name="position" />
+            <state_interface name="position" />
+        </joint>
+        <joint name="s1_joint_motor_06">
+            <command_interface name="position" />
+            <state_interface name="position" />
+        </joint>
         <!-- ****************** 1号从臂的转动关节 ****************** -->
         <joint name="s1_j01_base">
@@ -89,4 +97,12 @@
         </joint>
         <joint name="s2_joint_motor_04">
+            <command_interface name="position" />
+            <state_interface name="position" />
+        </joint>
+        <joint name="s2_joint_motor_05">
+            <command_interface name="position" />
+            <state_interface name="position" />
+        </joint>
+        <joint name="s2_joint_motor_06">
             <command_interface name="position" />
             <state_interface name="position" />
