Commit message: 蛇骨齿轮外啮合已完成，rviz表现完美

File: src/leonardo_description/psm_description/10_snake/11_snake_joints.xacro (robot description, xacro)
@@ -2,19 +2,11 @@
 <!-- 蛇形机械臂关节定义：适配 22 个 link，统一关节命名 -->
 <robot xmlns:xacro="http://www.ros.org/wiki/xacro">
-    <!-- ==========  X 轴偏移量  ========== -->
-    <xacro:property name="y_offset_01_02" value="0.051" />
-    <xacro:property name="y_offset_02_03" value="0.001" />
-    <xacro:property name="y_offset_03_04" value="0.004" />
-    <xacro:property name="y_offset_04_05" value="0.004" />
+    <!-- ==========  y轴偏移量  ========== -->
+    <xacro:property name="y_offset_01_02" value="0.0514" />
+    <xacro:property name="y_offset_02_03" value="0.0013" />
     <xacro:property name="y_offset_05_06" value="0.0084" />
     <xacro:property name="y_offset_06_07" value="0.0084" />
-    <xacro:property name="y_offset_07_08" value="0.004" />
-    <xacro:property name="y_offset_08_09" value="0.004" />
     <xacro:property name="y_offset_09_10" value="0.0055" />
     <xacro:property name="y_offset_10_11" value="0.0" />
-    <xacro:property name="y_offset_11_12" value="0.004" />
-    <xacro:property name="y_offset_12_13" value="0.004" />
-    <xacro:property name="y_offset_13_14" value="0.004" />
-    <xacro:property name="y_offset_14_15" value="0.004" />
     <xacro:property name="y_offset_15_16" value="0.0015" />
     <xacro:property name="y_offset_16_17" value="0.01172" />
@@ -24,11 +16,26 @@
     <xacro:property name="y_offset_20_21" value="0.0" />
     <xacro:property name="y_offset_20_22" value="0.0" />
-    <!-- 公转半径：两齿轮中心距（两齿轮半径之和） -->
+    <!-- 蛇骨公转半径：两齿轮中心距（两齿轮半径之和） -->
     <xacro:property name="orbit_r" value="0.0025" />
-    <!-- 公转角度限位（±45°） -->
+    <!-- 蛇骨公转角度限位（±45°） -->
     <xacro:property name="orbit_lower" value="${-pi/8.0}" />
     <xacro:property name="orbit_upper" value="${pi/8.0}" />
-    <!-- 原点相对齿轮中心的偏移 -->
-    <xacro:property name="origin_gear_center" value="0.00145" />
+    <!-- 蛇骨自身原点相对自身齿轮中心的偏移 -->
+    <xacro:property name="origin_gear_center_03_L" value="0.0" />
+    <xacro:property name="origin_gear_center_04_R" value="0.00145" />
+    <xacro:property name="origin_gear_center_04_L" value="0.0" />
+    <xacro:property name="origin_gear_center_05_R" value="0.00145" />
+    <xacro:property name="origin_gear_center_07_L" value="0.00145" />
+    <xacro:property name="origin_gear_center_08_R" value="0.0" />
+    <xacro:property name="origin_gear_center_08_L" value="0.00145" />
+    <xacro:property name="origin_gear_center_09_R" value="0.0" />
+    <xacro:property name="origin_gear_center_11_L" value="0.0" />
+    <xacro:property name="origin_gear_center_12_R" value="0.00145" />
+    <xacro:property name="origin_gear_center_12_L" value="0.0" />
+    <xacro:property name="origin_gear_center_13_R" value="0.00145" />
+    <xacro:property name="origin_gear_center_13_L" value="0.0" />
+    <xacro:property name="origin_gear_center_14_R" value="0.00145" />
+    <xacro:property name="origin_gear_center_14_L" value="0.0" />
+    <xacro:property name="origin_gear_center_15_R" value="0.00145" />
     <!-- ========= 最大力矩 ======== -->
     <xacro:property name="effort" value="1000" />
@@ -37,5 +44,5 @@
     <!-- ========== 宏定义：生成所有关节 ========== -->
     <xacro:macro name="get_snake_joints" params="prefix">
-        <!-- **************************  link01 -> link02  ************************** -->
+        <!-- ****************************************  link01 -> link02  **************************************** -->
         <joint name="${prefix}_joint_01_02" type="fixed">
             <parent link="${prefix}_01" />
@@ -43,5 +50,5 @@
             <origin xyz="0 ${y_offset_01_02} 0" rpy="0 0 0" />
         </joint>
-        <!-- **************************  link02 -> link03  ************************** -->
+        <!-- ****************************************  link02 -> link03  **************************************** -->
         <joint name="${prefix}_joint_02_03" type="fixed">
             <parent link="${prefix}_02" />
@@ -49,5 +56,5 @@
             <origin xyz="0 ${y_offset_02_03} 0" rpy="0 0 0" />
         </joint>
-        <!-- **************************  link03 -> link04  ************************** -->
+        <!-- ****************************************  link03 -> link04  **************************************** -->
         <link name="${prefix}_orbit_carrier_03" />
         <link name="${prefix}_gear_center_04" />
@@ -56,7 +63,8 @@
             <parent link="${prefix}_03" />
             <child link="${prefix}_orbit_carrier_03" />
-            <origin xyz="0 0 0" rpy="0 0 0" />
-            <axis xyz="0 0 1" />
-            <limit effort="${effort}" velocity="${velocity}" lower="${orbit_lower}" upper="${orbit_upper}" />
+            <origin xyz="0 ${origin_gear_center_03_L} 0" rpy="0 0 0" />
+            <axis xyz="0 0 1" />
+            <limit effort="${effort}" velocity="${velocity}"
+                lower="${orbit_lower}" upper="${orbit_upper}" />
         </joint>
         <!-- 自转关节：公转载体 -> link04 齿轮中心 -->
@@ -74,15 +82,30 @@
             <parent link="${prefix}_gear_center_04" />
             <child link="${prefix}_04" />
-            <origin xyz="0 ${origin_gear_center} 0" rpy="0 0 0" />
-        </joint>
-        <!-- **************************  link04 -> link05  ************************** -->
-        <joint name="${prefix}_joint_04_05" type="revolute">
+            <origin xyz="0 ${origin_gear_center_04_R} 0" rpy="0 0 0" />
+        </joint>
+        <!-- ****************************************  link04 -> link05  **************************************** -->
+        <link name="${prefix}_orbit_carrier_04" />
+        <link name="${prefix}_gear_center_05" />
+        <joint name="${prefix}_joint_04_orbit_carrier" type="revolute">
             <parent link="${prefix}_04" />
+            <child link="${prefix}_orbit_carrier_04" />
+            <origin xyz="0 ${origin_gear_center_04_L} 0" rpy="0 0 0" />
+            <axis xyz="1 0 0" />
+            <limit effort="${effort}" velocity="${velocity}" lower="${orbit_lower}" upper="${orbit_upper}" />
+        </joint>
+        <joint name="${prefix}_joint_05_spin" type="continuous">
+            <parent link="${prefix}_orbit_carrier_04" />
+            <child link="${prefix}_gear_center_05" />
+            <origin xyz="0 ${orbit_r} 0" rpy="0 0 0" />
+            <axis xyz="1 0 0" />
+            <limit effort="${effort}" velocity="${velocity}" />
+            <mimic joint="${prefix}_joint_04_orbit_carrier" multiplier="1" offset="0" />
+        </joint>
+        <joint name="${prefix}_joint_05_mount" type="fixed">
+            <parent link="${prefix}_gear_center_05" />
             <child link="${prefix}_05" />
-            <origin xyz="0 ${y_offset_04_05} 0" rpy="0 0 0" />
-            <axis xyz="1 0 0" />
-            <limit effort="${effort}" velocity="${velocity}" lower="${-pi}" upper="${pi}" />
-        </joint>
-        <!-- link05 -> link06 -->
+            <origin xyz="0 ${origin_gear_center_05_R} 0" rpy="0 0 0" />
+        </joint>
+        <!-- ****************************************  link05 -> link06  **************************************** -->
         <joint name="${prefix}_joint_05_06" type="fixed">
             <parent link="${prefix}_05" />
@@ -90,5 +113,5 @@
             <origin xyz="0 ${y_offset_05_06} 0" rpy="0 0 0" />
         </joint>
-        <!-- link06 -> link07 -->
+        <!-- ****************************************  link06 -> link07  **************************************** -->
         <joint name="${prefix}_joint_06_07" type="fixed">
             <parent link="${prefix}_06" />
@@ -96,21 +119,51 @@
             <origin xyz="0 ${y_offset_06_07} 0" rpy="0 0 0" />
         </joint>
-        <!-- link07 -> link08 -->
-        <joint name="${prefix}_joint_07_08" type="revolute">
+        <!-- ****************************************  link07 -> link08  **************************************** -->
+        <link name="${prefix}_orbit_carrier_07" />
+        <link name="${prefix}_gear_center_08" />
+        <joint name="${prefix}_joint_07_orbit_carrier" type="revolute">
             <parent link="${prefix}_07" />
+            <child link="${prefix}_orbit_carrier_07" />
+            <origin xyz="0 ${origin_gear_center_07_L} 0" rpy="0 0 0" />
+            <axis xyz="1 0 0" />
+            <limit effort="${effort}" velocity="${velocity}" lower="${orbit_lower}" upper="${orbit_upper}" />
+        </joint>
+        <joint name="${prefix}_joint_08_spin" type="continuous">
+            <parent link="${prefix}_orbit_carrier_07" />
+            <child link="${prefix}_gear_center_08" />
+            <origin xyz="0 ${orbit_r} 0" rpy="0 0 0" />
+            <axis xyz="1 0 0" />
+            <limit effort="${effort}" velocity="${velocity}" />
+            <mimic joint="${prefix}_joint_07_orbit_carrier" multiplier="1" offset="0" />
+        </joint>
+        <joint name="${prefix}_joint_08_mount" type="fixed">
+            <parent link="${prefix}_gear_center_08" />
             <child link="${prefix}_08" />
-            <origin xyz="0 ${y_offset_07_08} 0" rpy="0 0 0" />
-            <axis xyz="1 0 0" />
-            <limit effort="${effort}" velocity="${velocity}" lower="${-pi}" upper="${pi}" />
-        </joint>
-        <!-- link08 -> link09 -->
-        <joint name="${prefix}_joint_08_09" type="revolute">
+            <origin xyz="0 ${origin_gear_center_08_R} 0" rpy="0 0 0" />
+        </joint>
+        <!-- ****************************************  link08 -> link09  **************************************** -->
+        <link name="${prefix}_orbit_carrier_08" />
+        <link name="${prefix}_gear_center_09" />
+        <joint name="${prefix}_joint_08_orbit_carrier" type="revolute">
             <parent link="${prefix}_08" />
+            <child link="${prefix}_orbit_carrier_08" />
+            <origin xyz="0 ${origin_gear_center_08_L} 0" rpy="0 0 0" />
+            <axis xyz="0 0 1" />
+            <limit effort="${effort}" velocity="${velocity}" lower="${orbit_lower}" upper="${orbit_upper}" />
+        </joint>
+        <joint name="${prefix}_joint_09_spin" type="continuous">
+            <parent link="${prefix}_orbit_carrier_08" />
+            <child link="${prefix}_gear_center_09" />
+            <origin xyz="0 ${orbit_r} 0" rpy="0 0 0" />
+            <axis xyz="0 0 1" />
+            <limit effort="${effort}" velocity="${velocity}" />
+            <mimic joint="${prefix}_joint_08_orbit_carrier" multiplier="1" offset="0" />
+        </joint>
+        <joint name="${prefix}_joint_09_mount" type="fixed">
+            <parent link="${prefix}_gear_center_09" />
             <child link="${prefix}_09" />
-            <origin xyz="0 ${y_offset_08_09} 0" rpy="0 0 0" />
-            <axis xyz="0 0 1" />
-            <limit effort="${effort}" velocity="${velocity}" lower="${-pi}" upper="${pi}" />
-        </joint>
-        <!-- link09 -> link10  -->
+            <origin xyz="0 ${origin_gear_center_09_R} 0" rpy="0 0 0" />
+        </joint>
+        <!-- ****************************************  link09 -> link10  **************************************** -->
         <joint name="${prefix}_joint_09_10" type="fixed">
             <parent link="${prefix}_09" />
@@ -118,5 +171,5 @@
             <origin xyz="0 ${y_offset_09_10} 0" rpy="0 0 0" />
         </joint>
-        <!-- link10 -> link11  -->
+        <!-- ****************************************  link10 -> link11  **************************************** -->
         <joint name="${prefix}_joint_10_11" type="fixed">
             <parent link="${prefix}_10" />
@@ -124,37 +177,97 @@
             <origin xyz="0 ${y_offset_10_11} 0" rpy="0 0 0" />
         </joint>
-        <!-- link11 -> link12  -->
-        <joint name="${prefix}_joint_11_12" type="revolute">
+        <!-- ****************************************  link11 -> link12  **************************************** -->
+        <link name="${prefix}_orbit_carrier_11" />
+        <link name="${prefix}_gear_center_12" />
+        <joint name="${prefix}_joint_11_orbit_carrier" type="revolute">
             <parent link="${prefix}_11" />
+            <child link="${prefix}_orbit_carrier_11" />
+            <origin xyz="0 ${origin_gear_center_11_L} 0" rpy="0 0 0" />
+            <axis xyz="0 0 1" />
+            <limit effort="${effort}" velocity="${velocity}" lower="${orbit_lower}" upper="${orbit_upper}" />
+        </joint>
+        <joint name="${prefix}_joint_12_spin" type="continuous">
+            <parent link="${prefix}_orbit_carrier_11" />
+            <child link="${prefix}_gear_center_12" />
+            <origin xyz="0 ${orbit_r} 0" rpy="0 0 0" />
+            <axis xyz="0 0 1" />
+            <limit effort="${effort}" velocity="${velocity}" />
+            <mimic joint="${prefix}_joint_11_orbit_carrier" multiplier="1" offset="0" />
+        </joint>
+        <joint name="${prefix}_joint_12_mount" type="fixed">
+            <parent link="${prefix}_gear_center_12" />
             <child link="${prefix}_12" />
-            <origin xyz="0 ${y_offset_11_12} 0" rpy="0 0 0" />
-            <axis xyz="0 0 1" />
-            <limit effort="${effort}" velocity="${velocity}" lower="${-pi}" upper="${pi}" />
-        </joint>
-        <!-- link12 -> link13 -->
-        <joint name="${prefix}_joint_12_13" type="revolute">
+            <origin xyz="0 ${origin_gear_center_12_R} 0" rpy="0 0 0" />
+        </joint>
+        <!-- ****************************************  link12 -> link13  **************************************** -->
+        <link name="${prefix}_orbit_carrier_12" />
+        <link name="${prefix}_gear_center_13" />
+        <joint name="${prefix}_joint_12_orbit_carrier" type="revolute">
             <parent link="${prefix}_12" />
+            <child link="${prefix}_orbit_carrier_12" />
+            <origin xyz="0 ${origin_gear_center_12_L} 0" rpy="0 0 0" />
+            <axis xyz="1 0 0" />
+            <limit effort="${effort}" velocity="${velocity}" lower="${orbit_lower}" upper="${orbit_upper}" />
+        </joint>
+        <joint name="${prefix}_joint_13_spin" type="continuous">
+            <parent link="${prefix}_orbit_carrier_12" />
+            <child link="${prefix}_gear_center_13" />
+            <origin xyz="0 ${orbit_r} 0" rpy="0 0 0" />
+            <axis xyz="1 0 0" />
+            <limit effort="${effort}" velocity="${velocity}" />
+            <mimic joint="${prefix}_joint_12_orbit_carrier" multiplier="1" offset="0" />
+        </joint>
+        <joint name="${prefix}_joint_13_mount" type="fixed">
+            <parent link="${prefix}_gear_center_13" />
             <child link="${prefix}_13" />
-            <origin xyz="0 ${y_offset_12_13} 0" rpy="0 0 0" />
-            <axis xyz="1 0 0" />
-            <limit effort="${effort}" velocity="${velocity}" lower="${-pi}" upper="${pi}" />
-        </joint>
-        <!-- link13 -> link14 -->
-        <joint name="${prefix}_joint_13_14" type="revolute">
+            <origin xyz="0 ${origin_gear_center_13_R} 0" rpy="0 0 0" />
+        </joint>
+        <!-- ****************************************  link13 -> link14  **************************************** -->
+        <link name="${prefix}_orbit_carrier_13" />
+        <link name="${prefix}_gear_center_14" />
+        <joint name="${prefix}_joint_13_orbit_carrier" type="revolute">
             <parent link="${prefix}_13" />
+            <child link="${prefix}_orbit_carrier_13" />
+            <origin xyz="0 ${origin_gear_center_13_L} 0" rpy="0 0 0" />
+            <axis xyz="0 0 1" />
+            <limit effort="${effort}" velocity="${velocity}" lower="${orbit_lower}" upper="${orbit_upper}" />
+        </joint>
+        <joint name="${prefix}_joint_14_spin" type="continuous">
+            <parent link="${prefix}_orbit_carrier_13" />
+            <child link="${prefix}_gear_center_14" />
+            <origin xyz="0 ${orbit_r} 0" rpy="0 0 0" />
+            <axis xyz="0 0 1" />
+            <limit effort="${effort}" velocity="${velocity}" />
+            <mimic joint="${prefix}_joint_13_orbit_carrier" multiplier="1" offset="0" />
+        </joint>
+        <joint name="${prefix}_joint_14_mount" type="fixed">
+            <parent link="${prefix}_gear_center_14" />
             <child link="${prefix}_14" />
-            <origin xyz="0 ${y_offset_13_14} 0" rpy="0 0 0" />
-            <axis xyz="0 0 1" />
-            <limit effort="${effort}" velocity="${velocity}" lower="${-pi}" upper="${pi}" />
-        </joint>
-        <!-- link14 -> link15 -->
-        <joint name="${prefix}_joint_14_15" type="revolute">
+            <origin xyz="0 ${origin_gear_center_14_R} 0" rpy="0 0 0" />
+        </joint>
+        <!-- ****************************************  link14 -> link15  **************************************** -->
+        <link name="${prefix}_orbit_carrier_14" />
+        <link name="${prefix}_gear_center_15" />
+        <joint name="${prefix}_joint_14_orbit_carrier" type="revolute">
             <parent link="${prefix}_14" />
+            <child link="${prefix}_orbit_carrier_14" />
+            <origin xyz="0 ${origin_gear_center_14_L} 0" rpy="0 0 0" />
+            <axis xyz="1 0 0" />
+            <limit effort="${effort}" velocity="${velocity}" lower="${orbit_lower}" upper="${orbit_upper}" />
+        </joint>
+        <joint name="${prefix}_joint_15_spin" type="continuous">
+            <parent link="${prefix}_orbit_carrier_14" />
+            <child link="${prefix}_gear_center_15" />
+            <origin xyz="0 ${orbit_r} 0" rpy="0 0 0" />
+            <axis xyz="1 0 0" />
+            <limit effort="${effort}" velocity="${velocity}" />
+            <mimic joint="${prefix}_joint_14_orbit_carrier" multiplier="1" offset="0" />
+        </joint>
+        <joint name="${prefix}_joint_15_mount" type="fixed">
+            <parent link="${prefix}_gear_center_15" />
             <child link="${prefix}_15" />
-            <origin xyz="0 ${y_offset_14_15} 0" rpy="0 0 0" />
-            <axis xyz="1 0 0" />
-            <limit effort="${effort}" velocity="${velocity}" lower="${-pi}" upper="${pi}" />
-        </joint>
-        <!-- link15 -> link16 -->
+            <origin xyz="0 ${origin_gear_center_15_R} 0" rpy="0 0 0" />
+        </joint>
+        <!-- ****************************************  link15 -> link16  **************************************** -->
         <joint name="${prefix}_joint_15_16" type="fixed">
             <parent link="${prefix}_15" />
@@ -162,5 +275,5 @@
             <origin xyz="0 ${y_offset_15_16} 0" rpy="0 0 0" />
         </joint>
-        <!-- link16 -> link17 -->
+        <!-- ****************************************  link16 -> link17  **************************************** -->
         <joint name="${prefix}_joint_16_17" type="fixed">
             <parent link="${prefix}_16" />
@@ -168,5 +281,5 @@
             <origin xyz="0 ${y_offset_16_17} 0" rpy="0 0 0" />
         </joint>
-        <!-- link17 -> link18 -->
+        <!-- ****************************************  link17 -> link18  **************************************** -->
         <joint name="${prefix}_joint_17_18" type="revolute">
             <parent link="${prefix}_17" />
@@ -174,7 +287,7 @@
             <origin xyz="0 ${y_offset_17_18} 0" rpy="0 0 0" />
             <axis xyz="0 1 0" />
-            <limit effort="${effort}" velocity="${velocity}" lower="${-pi}" upper="${pi}" />
-        </joint>
-        <!-- link18 -> link19 -->
+            <limit effort="${effort}" velocity="${velocity}" lower="${-pi/2.0}" upper="${pi/2.0}" />
+        </joint>
+        <!-- ****************************************  link18 -> link19  **************************************** -->
         <joint name="${prefix}_joint_18_19" type="fixed">
             <parent link="${prefix}_18" />
@@ -182,5 +295,5 @@
             <origin xyz="0 ${y_offset_18_19} 0" rpy="0 0 0" />
         </joint>
-        <!-- link19 -> link20 -->
+        <!-- ****************************************  link19 -> link20  **************************************** -->
         <joint name="${prefix}_joint_19_20" type="fixed">
             <parent link="${prefix}_19" />
@@ -194,5 +307,5 @@
             <origin xyz="0 ${y_offset_20_21} 0" rpy="0 0 0" />
             <axis xyz="0 0 1" />
-            <limit effort="${effort}" velocity="${velocity}" lower="0" upper="${pi/3.0}" />
+            <limit effort="${effort}" velocity="${velocity}" lower="0" upper="${pi/6.0}" />
         </joint>
         <!-- link20 -> link22 （镜像钳） -->
