Commit message: psm_can_hardware已完成接口导出部分

File: src/leonardo_description/psm_description/10_snake/11_snake_joints.xacro (robot description, xacro)
@@ -60,5 +60,5 @@
         <link name="${prefix}_gear_center_04" />
         <!-- 公转关节：link03 -> 公转载体 -->
-        <joint name="${prefix}_joint_03_orbit_carrier" type="revolute">
+        <joint name="${prefix}_j03_oc" type="revolute">
             <parent link="${prefix}_03" />
             <child link="${prefix}_orbit_carrier_03" />
@@ -76,5 +76,5 @@
             <axis xyz="0 0 1" />
             <limit effort="${effort}" velocity="${velocity}" />
-            <mimic joint="${prefix}_joint_03_orbit_carrier" multiplier="1" offset="0" />
+            <mimic joint="${prefix}_j03_oc" multiplier="1" offset="0" />
         </joint>
         <!-- 固定关节：link04 齿轮中心 -> link04 原点 -->
@@ -87,5 +87,5 @@
         <link name="${prefix}_orbit_carrier_04" />
         <link name="${prefix}_gear_center_05" />
-        <joint name="${prefix}_joint_04_orbit_carrier" type="revolute">
+        <joint name="${prefix}_j04_oc" type="revolute">
             <parent link="${prefix}_04" />
             <child link="${prefix}_orbit_carrier_04" />
@@ -100,5 +100,5 @@
             <axis xyz="1 0 0" />
             <limit effort="${effort}" velocity="${velocity}" />
-            <mimic joint="${prefix}_joint_04_orbit_carrier" multiplier="1" offset="0" />
+            <mimic joint="${prefix}_j04_oc" multiplier="1" offset="0" />
         </joint>
         <joint name="${prefix}_joint_05_mount" type="fixed">
@@ -122,5 +122,5 @@
         <link name="${prefix}_orbit_carrier_07" />
         <link name="${prefix}_gear_center_08" />
-        <joint name="${prefix}_joint_07_orbit_carrier" type="revolute">
+        <joint name="${prefix}_j07_oc" type="revolute">
             <parent link="${prefix}_07" />
             <child link="${prefix}_orbit_carrier_07" />
@@ -135,5 +135,5 @@
             <axis xyz="1 0 0" />
             <limit effort="${effort}" velocity="${velocity}" />
-            <mimic joint="${prefix}_joint_07_orbit_carrier" multiplier="1" offset="0" />
+            <mimic joint="${prefix}_j07_oc" multiplier="1" offset="0" />
         </joint>
         <joint name="${prefix}_joint_08_mount" type="fixed">
@@ -145,5 +145,5 @@
         <link name="${prefix}_orbit_carrier_08" />
         <link name="${prefix}_gear_center_09" />
-        <joint name="${prefix}_joint_08_orbit_carrier" type="revolute">
+        <joint name="${prefix}_j08_oc" type="revolute">
             <parent link="${prefix}_08" />
             <child link="${prefix}_orbit_carrier_08" />
@@ -158,5 +158,5 @@
             <axis xyz="0 0 1" />
             <limit effort="${effort}" velocity="${velocity}" />
-            <mimic joint="${prefix}_joint_08_orbit_carrier" multiplier="1" offset="0" />
+            <mimic joint="${prefix}_j08_oc" multiplier="1" offset="0" />
         </joint>
         <joint name="${prefix}_joint_09_mount" type="fixed">
@@ -180,5 +180,5 @@
         <link name="${prefix}_orbit_carrier_11" />
         <link name="${prefix}_gear_center_12" />
-        <joint name="${prefix}_joint_11_orbit_carrier" type="revolute">
+        <joint name="${prefix}_j11_oc" type="revolute">
             <parent link="${prefix}_11" />
             <child link="${prefix}_orbit_carrier_11" />
@@ -193,5 +193,5 @@
             <axis xyz="0 0 1" />
             <limit effort="${effort}" velocity="${velocity}" />
-            <mimic joint="${prefix}_joint_11_orbit_carrier" multiplier="1" offset="0" />
+            <mimic joint="${prefix}_j11_oc" multiplier="1" offset="0" />
         </joint>
         <joint name="${prefix}_joint_12_mount" type="fixed">
@@ -203,5 +203,5 @@
         <link name="${prefix}_orbit_carrier_12" />
         <link name="${prefix}_gear_center_13" />
-        <joint name="${prefix}_joint_12_orbit_carrier" type="revolute">
+        <joint name="${prefix}_j12_oc" type="revolute">
             <parent link="${prefix}_12" />
             <child link="${prefix}_orbit_carrier_12" />
@@ -216,5 +216,5 @@
             <axis xyz="1 0 0" />
             <limit effort="${effort}" velocity="${velocity}" />
-            <mimic joint="${prefix}_joint_12_orbit_carrier" multiplier="1" offset="0" />
+            <mimic joint="${prefix}_j12_oc" multiplier="1" offset="0" />
         </joint>
         <joint name="${prefix}_joint_13_mount" type="fixed">
@@ -226,5 +226,5 @@
         <link name="${prefix}_orbit_carrier_13" />
         <link name="${prefix}_gear_center_14" />
-        <joint name="${prefix}_joint_13_orbit_carrier" type="revolute">
+        <joint name="${prefix}_j13_oc" type="revolute">
             <parent link="${prefix}_13" />
             <child link="${prefix}_orbit_carrier_13" />
@@ -239,5 +239,5 @@
             <axis xyz="0 0 1" />
             <limit effort="${effort}" velocity="${velocity}" />
-            <mimic joint="${prefix}_joint_13_orbit_carrier" multiplier="1" offset="0" />
+            <mimic joint="${prefix}_j13_oc" multiplier="1" offset="0" />
         </joint>
         <joint name="${prefix}_joint_14_mount" type="fixed">
@@ -249,5 +249,5 @@
         <link name="${prefix}_orbit_carrier_14" />
         <link name="${prefix}_gear_center_15" />
-        <joint name="${prefix}_joint_14_orbit_carrier" type="revolute">
+        <joint name="${prefix}_j14_oc" type="revolute">
             <parent link="${prefix}_14" />
             <child link="${prefix}_orbit_carrier_14" />
@@ -262,5 +262,5 @@
             <axis xyz="1 0 0" />
             <limit effort="${effort}" velocity="${velocity}" />
-            <mimic joint="${prefix}_joint_14_orbit_carrier" multiplier="1" offset="0" />
+            <mimic joint="${prefix}_j14_oc" multiplier="1" offset="0" />
         </joint>
         <joint name="${prefix}_joint_15_mount" type="fixed">
@@ -282,5 +282,5 @@
         </joint>
         <!-- ****************************************  link17 -> link18  **************************************** -->
-        <joint name="${prefix}_joint_17_18" type="revolute">
+        <joint name="${prefix}_j17_18" type="revolute">
             <parent link="${prefix}_17" />
             <child link="${prefix}_18" />
@@ -302,5 +302,5 @@
         </joint>
         <!-- link20 -> link21 （主动钳） -->
-        <joint name="${prefix}_joint_20_21" type="revolute">
+        <joint name="${prefix}_j20_21" type="revolute">
             <parent link="${prefix}_20" />
             <child link="${prefix}_21" />
@@ -316,5 +316,5 @@
             <axis xyz="0 0 1" />
             <limit effort="${effort}" velocity="${velocity}" lower="${-pi/3.0}" upper="${0}" />
-            <mimic joint="${prefix}_joint_20_21" multiplier="-1.0" offset="0.0" />
+            <mimic joint="${prefix}_j20_21" multiplier="-1.0" offset="0.0" />
         </joint>
     </xacro:macro>

File: src/leonardo_description/psm_description/10_snake/88_snake_robot.ros2_control.xacro (robot description, xacro)
@@ -3,5 +3,5 @@
     <ros2_control name="PSMCan0Hardware" type="system">
         <hardware>
-            <plugin>psm_can_hardware/PSMCan0Hardware</plugin>
+            <plugin>psm_can_hardware/PSMCan0HardwareInterface</plugin>
             <!-- CAN 通道 -->
             <param name="can_interface">can0</param>
@@ -14,82 +14,82 @@
         </hardware>
         <!-- ****************** 1号从臂的转动关节 ****************** -->
-        <joint name="s1_joint_03_orbit_carrier">
+        <joint name="s1_j03_oc">
             <command_interface name="position" />
             <state_interface name="position" />
         </joint>
-        <joint name="s1_joint_04_orbit_carrier">
+        <joint name="s1_j04_oc">
             <command_interface name="position" />
             <state_interface name="position" />
         </joint>
-        <joint name="s1_joint_07_orbit_carrier">
+        <joint name="s1_j07_oc">
             <command_interface name="position" />
             <state_interface name="position" />
         </joint>
-        <joint name="s1_joint_08_orbit_carrier">
+        <joint name="s1_j08_oc">
             <command_interface name="position" />
             <state_interface name="position" />
         </joint>
-        <joint name="s1_joint_11_orbit_carrier">
+        <joint name="s1_j11_oc">
             <command_interface name="position" />
             <state_interface name="position" />
         </joint>
-        <joint name="s1_joint_12_orbit_carrier">
+        <joint name="s1_j12_oc">
             <command_interface name="position" />
             <state_interface name="position" />
         </joint>
-        <joint name="s1_joint_13_orbit_carrier">
+        <joint name="s1_j13_oc">
             <command_interface name="position" />
             <state_interface name="position" />
         </joint>
-        <joint name="s1_joint_14_orbit_carrier">
+        <joint name="s1_j14_oc">
             <command_interface name="position" />
             <state_interface name="position" />
         </joint>
-        <joint name="s1_joint_17_18">
+        <joint name="s1_j17_18">
             <command_interface name="position" />
             <state_interface name="position" />
         </joint>
-        <joint name="s1_joint_20_21">
+        <joint name="s1_j20_21">
             <command_interface name="position" />
             <state_interface name="position" />
         </joint>
         <!-- ****************** 2号从臂的转动关节 ****************** -->
-        <joint name="s2_joint_03_orbit_carrier">
+        <joint name="s2_j03_oc">
             <command_interface name="position" />
             <state_interface name="position" />
         </joint>
-        <joint name="s2_joint_04_orbit_carrier">
+        <joint name="s2_j04_oc">
             <command_interface name="position" />
             <state_interface name="position" />
         </joint>
-        <joint name="s2_joint_07_orbit_carrier">
+        <joint name="s2_j07_oc">
             <command_interface name="position" />
             <state_interface name="position" />
         </joint>
-        <joint name="s2_joint_08_orbit_carrier">
+        <joint name="s2_j08_oc">
             <command_interface name="position" />
             <state_interface name="position" />
         </joint>
-        <joint name="s2_joint_11_orbit_carrier">
+        <joint name="s2_j11_oc">
             <command_interface name="position" />
             <state_interface name="position" />
         </joint>
-        <joint name="s2_joint_12_orbit_carrier">
+        <joint name="s2_j12_oc">
             <command_interface name="position" />
             <state_interface name="position" />
         </joint>
-        <joint name="s2_joint_13_orbit_carrier">
+        <joint name="s2_j13_oc">
             <command_interface name="position" />
             <state_interface name="position" />
         </joint>
-        <joint name="s2_joint_14_orbit_carrier">
+        <joint name="s2_j14_oc">
             <command_interface name="position" />
             <state_interface name="position" />
         </joint>
-        <joint name="s2_joint_17_18">
+        <joint name="s2_j17_18">
             <command_interface name="position" />
             <state_interface name="position" />
         </joint>
-        <joint name="s2_joint_20_21">
+        <joint name="s2_j20_21">
             <command_interface name="position" />
             <state_interface name="position" />
@@ -98,5 +98,5 @@
     <ros2_control name="PSMCan1Hardware" type="system">
         <hardware>
-            <plugin>psm_can_hardware/PSMCan1Hardware</plugin>
+            <plugin>psm_can_hardware/PSMCan1HardwareInterface</plugin>
             <!-- CAN 通道 -->
             <param name="can_interface">can1</param>
@@ -108,41 +108,41 @@
         </hardware>
         <!-- ****************** 3号从臂的转动关节 ****************** -->
-        <joint name="s3_joint_03_orbit_carrier">
+        <joint name="s3_j03_oc">
             <command_interface name="position" />
             <state_interface name="position" />
         </joint>
-        <joint name="s3_joint_04_orbit_carrier">
+        <joint name="s3_j04_oc">
             <command_interface name="position" />
             <state_interface name="position" />
         </joint>
-        <joint name="s3_joint_07_orbit_carrier">
+        <joint name="s3_j07_oc">
             <command_interface name="position" />
             <state_interface name="position" />
         </joint>
-        <joint name="s3_joint_08_orbit_carrier">
+        <joint name="s3_j08_oc">
             <command_interface name="position" />
             <state_interface name="position" />
         </joint>
-        <joint name="s3_joint_11_orbit_carrier">
+        <joint name="s3_j11_oc">
             <command_interface name="position" />
             <state_interface name="position" />
         </joint>
-        <joint name="s3_joint_12_orbit_carrier">
+        <joint name="s3_j12_oc">
             <command_interface name="position" />
             <state_interface name="position" />
         </joint>
-        <joint name="s3_joint_13_orbit_carrier">
+        <joint name="s3_j13_oc">
             <command_interface name="position" />
             <state_interface name="position" />
         </joint>
-        <joint name="s3_joint_14_orbit_carrier">
+        <joint name="s3_j14_oc">
             <command_interface name="position" />
             <state_interface name="position" />
         </joint>
-        <joint name="s3_joint_17_18">
+        <joint name="s3_j17_18">
             <command_interface name="position" />
             <state_interface name="position" />
         </joint>
-        <joint name="s3_joint_20_21">
+        <joint name="s3_j20_21">
             <command_interface name="position" />
             <state_interface name="position" />

File: src/leonardo_description/urdf/leonardo.urdf.xacro (robot description, xacro)
@@ -1,14 +1,14 @@
 <?xml version="1.0"?>
 <robot xmlns:xacro="http://www.ros.org/wiki/xacro" name="leonardo">
-    <!-- ==================== 引入 MTM 双臂 ==================== -->
+    <!-- ==================== 引入 MTM 主手 ==================== -->
     <xacro:include
         filename="$(find leonardo_description)/mtm_description/urdf/fd_bimanual.config.xacro" />
-    <!-- ==================== 引入 FT3215  ==================== -->
-    <xacro:include filename="$(find leonardo_description)/ft3215_description/ft3215.urdf.xacro" />
-    <!-- ==================== 把 FT3215 挂到 fd_left_base 上 ==================== -->
-    <joint name="fd_left_base_to_ft3215" type="fixed">
+    <!-- ==================== 引入 PSM 从手  ==================== -->
+    <xacro:include filename="$(find leonardo_description)/psm_description/urdf/snakes.urdf.xacro" />
+    <!-- ==================== 把 PSM 从手 挂到 MTM 双手 上 ==================== -->
+    <joint name="MTM_PSM_base" type="fixed">
         <origin xyz="0 0 0" rpy="0 0 0" />
         <parent link="fd_left_base" />
-        <child link="link_ft_11" />
+        <child link="snakes_footprint" />
     </joint>
 </robot>
