Commit message: 准备把蛇臂模型顺着x轴

File: src/leonardo_description/mtm_description/urdf/fd_bimanual.urdf.xacro (robot description, xacro)
@@ -137,5 +137,5 @@
     <!-- ============================================================ -->
     <joint name="fd_left_to_right_base" type="fixed">
-        <origin rpy="0 0 0" xyz="0.1 0.0 0.0" />
+        <origin rpy="0 0 ${pi}" xyz="0 0.01 0.0" />
         <parent link="fd_left_base" />
         <child link="fd_right_base" />
@@ -146,5 +146,5 @@
     <ros2_control name="FDLeftHardware" type="system">
         <hardware>
-            <plugin>fd_left_hardware/FDLeftHardwareInterface</plugin>
+            <plugin>mtm_hardware_interface/FDLeftHardwareInterface</plugin>
             <param name="interface_id">-1</param>
             <param name="interface_serial_number">40819</param>
@@ -200,5 +200,5 @@
     <ros2_control name="FDRightHardware" type="system">
         <hardware>
-            <plugin>fd_right_hardware/FDRightHardwareInterface</plugin>
+            <plugin>mtm_hardware_interface/FDRightHardwareInterface</plugin>
             <param name="interface_id">-1</param>
             <param name="interface_serial_number">40619</param>

File: src/leonardo_description/psm_description/10_snake/10_snake_links.xacro (robot description, xacro)
@@ -301,5 +301,5 @@
                     <mesh filename="${stl_path}/17.stl" scale="${mesh_scale}" />
                 </geometry>
-                <origin xyz="0 0 0" rpy="0 0 ${pi/2.0}" />
+                <origin xyz="0 0 0" rpy="0 0 ${pi/2}" />
                 <material name="${prefix}_link17" />
             </visual>

File: src/leonardo_description/psm_description/10_snake/69_snake_robot.xacro (robot description, xacro)
@@ -24,18 +24,24 @@
     <!-- 17 生成 base_footprint_snake 固定基座 -->
     <link name="base_footprint_snake" />
-    <joint name="base_s1_link01" type="fixed">
+    <joint name="s1_j01_base" type="prismatic">
         <parent link="base_footprint_snake" />
         <child link="s1_01" />
         <origin xyz="0 0 0" rpy="0 0 0" />
+        <axis xyz="0 1 0" />
+        <limit effort="10.0" velocity="0.5" lower="-0.1" upper="0.1" />
     </joint>
-    <joint name="base_s2_link01" type="fixed">
+    <joint name="s2_j01_base" type="prismatic">
         <parent link="base_footprint_snake" />
         <child link="s2_01" />
         <origin xyz="0.05 0 0" rpy="0 0 0" />
+        <axis xyz="0 1 0" />
+        <limit effort="10.0" velocity="0.5" lower="-0.1" upper="0.1" />
     </joint>
-    <joint name="base_s3_link01" type="fixed">
+    <joint name="s3_j01_base" type="prismatic">
         <parent link="base_footprint_snake" />
         <child link="s3_01" />
-        <origin xyz="-0.05 0 0" rpy="0 0 0" />
+        <origin xyz="0.1 0 0" rpy="0 0 0" />
+        <axis xyz="0 1 0" />
+        <limit effort="10.0" velocity="0.5" lower="-0.1" upper="0.1" />
     </joint>
 </robot>

File: src/leonardo_description/psm_description/10_snake/88_snake_robot.ros2_control.xacro (robot description, xacro)
@@ -14,21 +14,25 @@
         </hardware>
         <!-- ****************** 1号从臂的电机 ****************** -->
-        <joint name="s1__joint_motor_01">
-            <command_interface name="position" />
-            <state_interface name="position" />
-        </joint>
-        <joint name="s1__joint_motor_02">
-            <command_interface name="position" />
-            <state_interface name="position" />
-        </joint>
-        <joint name="s1__joint_motor_03">
-            <command_interface name="position" />
-            <state_interface name="position" />
-        </joint>
-        <joint name="s1__joint_motor_04">
+        <joint name="s1_joint_motor_01">
+            <command_interface name="position" />
+            <state_interface name="position" />
+        </joint>
+        <joint name="s1_joint_motor_02">
+            <command_interface name="position" />
+            <state_interface name="position" />
+        </joint>
+        <joint name="s1_joint_motor_03">
+            <command_interface name="position" />
+            <state_interface name="position" />
+        </joint>
+        <joint name="s1_joint_motor_04">
             <command_interface name="position" />
             <state_interface name="position" />
         </joint>
         <!-- ****************** 1号从臂的转动关节 ****************** -->
+        <joint name="s1_j01_base">
+            <command_interface name="position" />
+            <state_interface name="position" />
+        </joint>
         <joint name="s1_j03_oc">
             <command_interface name="position" />
@@ -72,21 +76,25 @@
         </joint>
         <!-- ****************** 1号从臂的电机 ****************** -->
-        <joint name="s2__joint_motor_01">
-            <command_interface name="position" />
-            <state_interface name="position" />
-        </joint>
-        <joint name="s2__joint_motor_02">
-            <command_interface name="position" />
-            <state_interface name="position" />
-        </joint>
-        <joint name="s2__joint_motor_03">
-            <command_interface name="position" />
-            <state_interface name="position" />
-        </joint>
-        <joint name="s2__joint_motor_04">
+        <joint name="s2_joint_motor_01">
+            <command_interface name="position" />
+            <state_interface name="position" />
+        </joint>
+        <joint name="s2_joint_motor_02">
+            <command_interface name="position" />
+            <state_interface name="position" />
+        </joint>
+        <joint name="s2_joint_motor_03">
+            <command_interface name="position" />
+            <state_interface name="position" />
+        </joint>
+        <joint name="s2_joint_motor_04">
             <command_interface name="position" />
             <state_interface name="position" />
         </joint>
         <!-- ****************** 2号从臂的转动关节 ****************** -->
+        <joint name="s2_j01_base">
+            <command_interface name="position" />
+            <state_interface name="position" />
+        </joint>
         <joint name="s2_j03_oc">
             <command_interface name="position" />
@@ -142,21 +150,25 @@
         </hardware>
         <!-- ****************** 3号从臂的电机 ****************** -->
-        <joint name="s3__joint_motor_01">
-            <command_interface name="position" />
-            <state_interface name="position" />
-        </joint>
-        <joint name="s3__joint_motor_02">
-            <command_interface name="position" />
-            <state_interface name="position" />
-        </joint>
-        <joint name="s3__joint_motor_03">
-            <command_interface name="position" />
-            <state_interface name="position" />
-        </joint>
-        <joint name="s3__joint_motor_04">
+        <joint name="s3_joint_motor_01">
+            <command_interface name="position" />
+            <state_interface name="position" />
+        </joint>
+        <joint name="s3_joint_motor_02">
+            <command_interface name="position" />
+            <state_interface name="position" />
+        </joint>
+        <joint name="s3_joint_motor_03">
+            <command_interface name="position" />
+            <state_interface name="position" />
+        </joint>
+        <joint name="s3_joint_motor_04">
             <command_interface name="position" />
             <state_interface name="position" />
         </joint>
         <!-- ****************** 3号从臂的转动关节 ****************** -->
+        <joint name="s3_j01_base">
+            <command_interface name="position" />
+            <state_interface name="position" />
+        </joint>
         <joint name="s3_j03_oc">
             <command_interface name="position" />

File: src/leonardo_description/urdf/leonardo.urdf.xacro (robot description, xacro)
@@ -1,8 +1,8 @@
 <?xml version="1.0"?>
 <robot xmlns:xacro="http://www.ros.org/wiki/xacro" name="leonardo">
-    <!-- ==================== 引入 MTM 主手 ==================== -->
+    <!-- ==================== 引入 fd 主手 ==================== -->
     <xacro:include
-        filename="$(find leonardo_description)/mtm_description/urdf/fd_bimanual.config.xacro" />
-    <!-- ==================== 引入 PSM 从手  ==================== -->
+        filename="$(find leonardo_description)/mtm_description/urdf/fd_bimanual.urdf.xacro" />
+    <!-- ==================== 引入 snake 从手  ==================== -->
     <xacro:include filename="$(find leonardo_description)/psm_description/urdf/snakes.urdf.xacro" />
     <!-- ==================== 把 PSM 从手 挂到 MTM 双手 上 ==================== -->

Commit message: 卡在运动学算法上了

File: src/leonardo_description/mtm_description/urdf/fd_bimanual.urdf.xacro (robot description, xacro)
@@ -137,5 +137,5 @@
     <!-- ============================================================ -->
     <joint name="fd_left_to_right_base" type="fixed">
-        <origin rpy="0 0 ${pi}" xyz="0 0.01 0.0" />
+        <origin rpy="0 0 0" xyz="0 0.1 0.0" />
         <parent link="fd_left_base" />
         <child link="fd_right_base" />
