Commit message: 准备改造踏板发布器——PedalPublisher，改造成生命周期节点

File: src/leonardo_description/psm_description/urdf/view_gear.urdf.xacro (robot description, xacro)
@@ -8,5 +8,5 @@
     <link name="gear1_link">
         <visual>
-            <origin xyz="0 0 0" rpy="0 0 0" />
+            <origin xyz="0 0 -${width/2.0}" rpy="0 0 0" />
             <geometry>
                 <cylinder radius="${r}" length="${width}" />
@@ -33,5 +33,5 @@
     <link name="gear2_link">
         <visual>
-            <origin xyz="0 0 0" rpy="0 0 0" />
+            <origin xyz="0 0 -${width/2.0}" rpy="0 0 0" />
             <geometry>
                 <cylinder radius="${r}" length="${width}" />
